Commit message: base driver now uses third party wrapper, description files cleaned to some degree, gamepad controller support added

File: poli_description/urdf/accessories.urdf.xacro (robot description, xacro)
@@ -22,85 +22,12 @@
 -->
 <robot name="segway_accessories" xmlns:xacro="http://ros.org/wiki/xacro">
-    <xacro:include filename="$(find poli_description)/urdf/sensors/rgbd_sensor.urdf.xacro"/>
-    <xacro:include filename="$(find poli_description)/urdf/sensors/sick_tim.urdf.xacro"/>
     <xacro:include filename="$(find poli_description)/urdf/sensors/hokuyo_ust20lx.urdf.xacro"/>
-    <xacro:include filename="$(find poli_description)/urdf/sensors/velodyne_vlp16.urdf.xacro"/>
-    <xacro:include filename="$(find poli_description)/urdf/sensors/pgr_flea3.urdf.xacro"/>
     <property name="M_PI" value="3.14159"/>
     <xacro:macro name="segway_accessories">
-        <!-- CH Robotics UM7 Link-->
-        <xacro:if value="$(optenv SEGWAY_HAS_EXT_IMU false)">
-            <link name="ext_imu_frame"/>
-            <joint name="ext_imu_joint" type="fixed">
-                <origin xyz="$(optenv EXT_IMU_XYZ 0 0 0.30635)" rpy="$(optenv EXT_IMU_RPY 0 0 0)" />
-                <parent link="$(optenv SEGWAY_PARENT_LINK base_chassis_link)" />
-                <child link="ext_imu_frame" />
-            </joint>
-            <gazebo>
-                <plugin name="imu_controller" filename="libhector_gazebo_ros_imu.so">
-                    <alwaysOn>1</alwaysOn>
-                    <updateRate>50.0</updateRate>
-                    <bodyName>ext_imu_frame</bodyName>
-                    <topicName>/segway/feedback/ext_imu</topicName>
-                    <accelDrift>0.005 0.005 0.005</accelDrift>
-                    <accelGaussianNoise>0.005 0.005 0.005</accelGaussianNoise>
-                    <rateDrift>0.005 0.005 0.005 </rateDrift>
-                    <rateGaussianNoise>0.005 0.005 0.005 </rateGaussianNoise>
-                    <headingDrift>0.005</headingDrift>
-                    <headingGaussianNoise>0.005</headingGaussianNoise>
-                </plugin>
-            </gazebo>
-        </xacro:if>
-        <!--GPS Link-->
-        <xacro:if value="$(optenv SEGWAY_HAS_GPS false)">
-            <link name="gps_frame"/>
-            <joint name="gps_joint" type="fixed">
-                <origin xyz="$(optenv GPS_XYZ -0.1189 0 0.34665)" rpy="$(optenv GPS_RPY 0 0 0)" />
-                <parent link="$(optenv SEGWAY_PARENT_LINK base_chassis_link)" />
-                <child link="gps_frame" />
-            </joint>
-            <gazebo>
-                <plugin name="gps_controller" filename="libhector_gazebo_ros_gps.so">
-                    <alwaysOn>1</alwaysOn>
-                    <updateRate>40</updateRate>
-                    <bodyName>gps_frame</bodyName>
-                    <topicName>/segway/feedback/gps/fix_2d</topicName>
-                    <velocityTopicName>/segway/feedback/gps/vel</velocityTopicName>
-                    <referenceLatitude>40.712784</referenceLatitude>
-                    <referenceLongitude>-74.005941</referenceLongitude>
-                    <referenceHeading>0</referenceHeading>
-                    <referenceAltitude>0</referenceAltitude>
-                    <drift>0.0001 0.0001 0.0001</drift>
-                </plugin>
-            </gazebo>
-        </xacro:if>
-        <!-- RGBD Sensor -->
-        <xacro:if value="$(optenv SEGWAY_HAS_KINECT false)">
-            <xacro:rgbd_sensor rgbd_prefix="rgbd" parent="$(optenv SEGWAY_PARENT_LINK base_chassis_link)">
-                <origin xyz="$(optenv RGBD_SENSOR_XYZ 0 0 1.0)" rpy="$(optenv RGBD_SENSOR_RPY 0 0 3.1416)" />
-            </xacro:rgbd_sensor>
-        </xacro:if>
-        <!-- First laser Sensor -->
-        <xacro:if value="$(optenv SEGWAY_HAS_ONE_2D_LASER false)">
-            <!-- SICK TIM Sensor -->
-            <xacro:if value="$(optenv SEGWAY_LASER1_IS_SICK_TIM false)">
-                <xacro:sick_tim laser_prefix="$(optenv LASER1_PREFIX base)" parent="$(optenv SEGWAY_PARENT_LINK base_chassis_link)">
-                    <origin xyz="$(optenv LASER1_XYZ 0.35 0 0.2)" rpy="$(optenv LASER1_RPY 3.14159 0 0)" />
-                </xacro:sick_tim>
-            </xacro:if>
-            <xacro:if value="$(optenv SEGWAY_LASER1_IS_HOKUYO false)">
-                <xacro:hokuyo_ust20lx laser_prefix="$(optenv LASER1_PREFIX base)" parent="$(optenv VECTOR_PARENT_LINK base_chassis_link)">
-                    <origin xyz="$(optenv LASER1_XYZ 0.35 0 0.2)" rpy="$(optenv LASER1_RPY 3.14159 0 0)" />
-                </xacro:hokuyo_ust20lx>
-            </xacro:if>
-        </xacro:if>
+	<xacro:hokuyo_ust20lx laser_prefix="$(optenv LASER1_PREFIX base)" parent="$(optenv VECTOR_PARENT_LINK base_chassis_link)">
+	 <origin xyz="$(optenv LASER1_XYZ 0.35 0 0.2)" rpy="$(optenv LASER1_RPY 3.14159 0 0)" />
+	</xacro:hokuyo_ust20lx>
         <!-- Second laser Sensor -->
         <xacro:if value="$(optenv SEGWAY_HAS_SECOND_2D_LASER false)">
-            <!-- SICK TIM Sensor -->
-            <xacro:if value="$(optenv SEGWAY_LASER2_IS_SICK_TIM false)">
-                <xacro:sick_tim laser_prefix="$(optenv LASER2_PREFIX base)" parent="$(optenv SEGWAY_PARENT_LINK base_chassis_link)">
-                    <origin xyz="$(optenv LASER2_XYZ 0.35 0 0.2)" rpy="$(optenv LASER2_RPY 3.14159 0 0)" />
-                </xacro:sick_tim>
-            </xacro:if>
             <xacro:if value="$(optenv SEGWAY_LASER2_IS_HOKUYO false)">
                 <xacro:hokuyo_ust20lx laser_prefix="$(optenv LASER2_PREFIX base)" parent="$(optenv VECTOR_PARENT_LINK base_chassis_link)">
@@ -109,19 +36,4 @@
             </xacro:if>
         </xacro:if>
-        <!-- Velodyne VLP-16 Sensor -->
-        <xacro:if value="$(optenv SEGWAY_HAS_VLP16 false)">
-            <xacro:velodyne_vlp16 parent="$(optenv SEGWAY_PARENT_LINK base_chassis_link)">
-                <origin xyz="$(optenv VLP16_XYZ 0 0 0.39991)" rpy="$(optenv VLP16_RPY 0 0 0)" />
-            </xacro:velodyne_vlp16>
-        </xacro:if>
-        <!-- PGR FLEA3 Sensor -->
-        <xacro:if value="$(optenv SEGWAY_HAS_FLEA3 false)">
-            <xacro:pgr_flea3 camera_prefix="camera" parent="$(optenv SEGWAY_PARENT_LINK base_chassis_link)"
-                          image_format="R8G8B8" image_topic_name="image_raw"
-                          camera_info_topic_name="camera_info" hfov="90" focal_length="317.772992"
-                          hack_baseline="0" image_width="640" image_height="480">
-                <origin xyz="$(optenv FLEA3_XYZ 0 0 0.32739)" rpy="$(optenv FLEA3_RPY 0 0 0)" />
-            </xacro:pgr_flea3>
-        </xacro:if>
     </xacro:macro>
 </robot>
