Commit message: added meshes of basic components. baseplate is added and positioned correctly

File: poli_description/robots/poli.urdf.xacro (robot description, xacro)
@@ -1,5 +1,108 @@
 <?xml version="1.0"?>
+<!--
+Software License Agreement (BSD)
+Copyright (c) 2017, University of Texas Austin
+Author Maxwell Svetlik
+Redistribution and use in source and binary forms, with or without modification, are permitted provided that
+the following conditions are met:
+ * Redistributions of source code must retain the above copyright notice, this list of conditions and the
+   following disclaimer.
+ * Redistributions in binary form must reproduce the above copyright notice, this list of conditions and the
+   following disclaimer in the documentation and/or other materials provided with the distribution.
+ * Neither the name of Stanley Innovation, Inc. nor the names of its contributors may be used to endorse or promote
+   products derived from this software without specific prior written permission.
+THIS SOFTWARE IS PROVIDED BY THE COPYRIGHT HOLDERS AND CONTRIBUTORS "AS IS" AND ANY EXPRESS OR IMPLIED WAR-
+RANTIES, INCLUDING, BUT NOT LIMITED TO, THE IMPLIED WARRANTIES OF MERCHANTABILITY AND FITNESS FOR A PARTICULAR
+PURPOSE ARE DISCLAIMED. IN NO EVENT SHALL THE COPYRIGHT HOLDER OR CONTRIBUTORS BE LIABLE FOR ANY DIRECT, IN-
+DIRECT, INCIDENTAL, SPECIAL, EXEMPLARY, OR CONSEQUENTIAL DAMAGES (INCLUDING, BUT NOT LIMITED TO, PROCUREMENT
+OF SUBSTITUTE GOODS OR SERVICES; LOSS OF USE, DATA, OR PROFITS; OR BUSINESS INTERRUPTION) HOWEVER CAUSED AND
+ON ANY THEORY OF LIABILITY, WHETHER IN CONTRACT, STRICT LIABILITY, OR TORT (INCLUDING NEGLIGENCE OR OTHERWISE)
+ARISING IN ANY WAY OUT OF THE USE OF THIS SOFTWARE, EVEN IF ADVISED OF THE POSSIBILITY OF SUCH DAMAGE.
+-->
 <robot name="segway_robot" xmlns:xacro="http://ros.org/wiki/xacro">
-  <xacro:include filename="$(find poli_description)/urdf/RMP_110/rmp.urdf.xacro" />
-  <xacro:segway_robot />
+    <!-- Included URDF/XACRO Files -->
+    <xacro:include filename="$(find poli_description)/urdf/segway_components/battery.urdf.xacro" />
+    <xacro:include filename="$(find poli_description)/urdf/segway_components/i2_wheel.urdf.xacro" />
+    <xacro:include filename="$(find poli_description)/urdf/segway_components/caster_assembly_110.urdf.xacro" />
+    <xacro:include filename="$(find poli_description)/urdf/segway_components/powerbase_110.urdf.xacro" />
+    <xacro:include filename="$(find poli_description)/urdf/segway_components/hmi_box_110.urdf.xacro" />
+    <xacro:include filename="$(find poli_description)/urdf/segway_components/hmi_plate_110.urdf.xacro" />
+    <xacro:include filename="$(find poli_description)/urdf/accessories.urdf.xacro" />
+    <xacro:include filename="$(find poli_description)/urdf/poli_components/base_plate.urdf.xacro"/>
+    <property name="M_PI" value="3.14159"/>
+    <property name="HALF_PI" value="1.57079"/>
+    <!-- Wheel Mounting Positions -->
+    <xacro:property name="track" value="0.48122440" />
+    <xacro:property name="wheel_vertical_offset" value="0.08255015" />
+    <!-- Wheel Properties -->
+    <xacro:property name="wheel_length" value="0.09224900" />
+    <xacro:property name="wheel_radius" value="0.2405681" />
+    <xacro:macro name="segway_robot">
+        <gazebo>
+          <plugin name="gazebo_ros_control" filename="libgazebo_ros_control.so">
+              <robotNamespace>/</robotNamespace>
+          </plugin>
+        </gazebo>
+        <!-- Base link is the center of the robot's chassis between the motors projected on the ground -->
+        <link name="base_link"/>
+        <!--Chassis -->
+        <xacro:powerbase_110 chassis_prefix="base" parent="base_link">
+            <origin xyz="0 0 ${-wheel_vertical_offset + wheel_radius}" rpy="0 0 0" />
+        </xacro:powerbase_110>
+        <link name="inertial_collision_link">
+			<inertial>
+				<mass value="29.756375" />
+				<origin xyz="0.001751 0.000008 0.018544" />
+				<inertia ixx="0.696269"  ixy="0.016133" ixz="0.003232"
+                         iyx="0.016133"  iyy="0.299110" iyz="-0.000004"
+                         izx="-0.077476" izy="-0.000004" izz="0.864394" />
+			</inertial>
+            <collision>
+				<geometry>
+					<mesh filename="package://poli_description/meshes/collision/110_powerbase_collision.stl" />
+				</geometry>
+			</collision>
+		</link>
+		<joint name="inertial_collision_joint" type="fixed" >
+		    <parent link="base_chassis_link" />
+		    <child link="inertial_collision_link" />
+		</joint>
+        <!-- Propulsion Batteries -->
+        <xacro:battery battery_prefix="mcu_1" parent="base_chassis_link">
+            <origin xyz="-0.09298 0 0" rpy="0 0 0" />
+        </xacro:battery>
+        <!-- Aux Batteries -->
+        <xacro:battery battery_prefix="aux" parent="base_chassis_link">
+            <origin xyz="0.09298 0 0" rpy="0 0 ${M_PI}" />
+        </xacro:battery>
+        <!-- HMI Box -->
+        <xacro:hmi_box_110 parent="base_chassis_link">
+            <origin xyz="0 0 0.09504494" rpy="0 0 0" />
+        </xacro:hmi_box_110>
+        <xacro:hmi_plate_110 parent="hmi_link">
+            <origin xyz="0 0 0" rpy="0 0 0" />
+        </xacro:hmi_plate_110>
+        <!-- Segway wheel macros -->
+        <xacro:i2_wheel wheel_prefix="left" parent="base_chassis_link" visual_rotation="0.0">
+            <origin xyz="0 ${track/2} ${wheel_vertical_offset}" rpy="0 0 0" />
+        </xacro:i2_wheel>
+        <xacro:i2_wheel wheel_prefix="right" parent="base_chassis_link" visual_rotation="${M_PI}">
+            <origin xyz="0 ${-track/2} ${wheel_vertical_offset}" rpy="0 0 0" />
+        </xacro:i2_wheel>
+        <!-- Segway Caster Assembly-->
+        <xacro:caster_assembly_110 caster_prefix="rear" parent="base_chassis_link">
+            <origin xyz="-0.32784550 0 0.03326933" rpy="0 0 ${M_PI}" />
+        </xacro:caster_assembly_110>
+        <xacro:caster_assembly_110 caster_prefix="front" parent="base_chassis_link">
+            <origin xyz="0.32784550 0 0.03326933" rpy="0 0 0" />
+        </xacro:caster_assembly_110>
+        <!-- Setup any accessories defined in the environment -->
+        <xacro:segway_accessories />
+        <xacro:base_plate parent="base_chassis_link">
+            <origin xyz="-0.0762 -0.15875 0.076" rpy="${HALF_PI} 0 ${HALF_PI}"/>
+        </xacro:base_plate>
+        <xacro:pillar_plate parent="base_plate_link">
+            <origin xyz="1 1 1" rpy="0 0 0"/>
+        </xacro:pillar_plate>
+    </xacro:macro>
 </robot>

Commit message: position changes for base plate. added pillar

File: poli_description/robots/poli.urdf.xacro (robot description, xacro)
@@ -30,4 +30,6 @@
     <xacro:include filename="$(find poli_description)/urdf/accessories.urdf.xacro" />
     <xacro:include filename="$(find poli_description)/urdf/poli_components/base_plate.urdf.xacro"/>
+    <xacro:include filename="$(find poli_description)/urdf/poli_components/pillar.urdf.xacro"/>
+    <xacro:include filename="$(find poli_description)/urdf/poli_components/pillar_plate.urdf.xacro"/>
     <property name="M_PI" value="3.14159"/>
     <property name="HALF_PI" value="1.57079"/>
@@ -100,9 +102,9 @@
         <xacro:segway_accessories />
         <xacro:base_plate parent="base_chassis_link">
-            <origin xyz="-0.0762 -0.15875 0.076" rpy="${HALF_PI} 0 ${HALF_PI}"/>
+            <origin xyz="-0.0762 -0.16355 0.076" rpy="${HALF_PI} 0 ${HALF_PI}"/>
         </xacro:base_plate>
-        <xacro:pillar_plate parent="base_plate_link">
-            <origin xyz="1 1 1" rpy="0 0 0"/>
-        </xacro:pillar_plate>
+        <xacro:pillar parent="base_plate_link">
+            <origin xyz="0.2275586 0 0" rpy="0 -${HALF_PI} 0"/>
+        </xacro:pillar>
     </xacro:macro>
 </robot>

Commit message: flipped baseplate to match reality. added telescope to pillar

File: poli_description/robots/poli.urdf.xacro (robot description, xacro)
@@ -102,8 +102,8 @@
         <xacro:segway_accessories />
         <xacro:base_plate parent="base_chassis_link">
-            <origin xyz="-0.0762 -0.16355 0.076" rpy="${HALF_PI} 0 ${HALF_PI}"/>
+            <origin xyz="0.0762 0.16355 0.076" rpy="${HALF_PI} 0 -${HALF_PI}"/>
         </xacro:base_plate>
         <xacro:pillar parent="base_plate_link">
-            <origin xyz="0.2275586 0 0" rpy="0 -${HALF_PI} 0"/>
+            <origin xyz="0.2315586 0 0.0075" rpy="0 -${HALF_PI} 0"/>
         </xacro:pillar>
     </xacro:macro>

File: poli_description/urdf/poli_components/pillar.urdf.xacro (robot description, xacro)
@@ -22,13 +22,32 @@
 <robot xmlns:xacro="http://ros.org/wiki/xacro" name="pillar">
     <xacro:macro name="pillar" params="parent *origin">
-        <joint name="pillar_joint" type="fixed">
+        <joint name="pillar_base_joint" type="fixed">
             <xacro:insert_block name="origin" />
             <parent link="${parent}" />
-            <child link="pillar_link" />
+            <child link="pillar_base_link" />
         </joint>
-        <link name="pillar_link">
+        <link name="pillar_base_link">
             <visual>
                 <geometry>
-                    <mesh filename="package://poli_description/meshes/components/pillar.STL" />
+                    <mesh filename="package://poli_description/meshes/components/pillar_exterior.STL" />
+                </geometry>
+            </visual>
+            <collision>
+                <geometry>
+                    <box size="0.1 0.1 0.1"/>
+                </geometry>
+            </collision>
+        </link>
+        <joint name="pillar_telescope_joint" type="prismatic">
+            <origin xyz="0.2175586 0.1 0.02" rpy="0 -1.570796 0"/>
+            <parent link="${parent}" />
+            <child link="pillar_telescope_link" />
+            <limit effort="30" velocity="1.0" lower="0.0" upper="0.4" />
+            <axis xyz="0 1 0"/>
+        </joint>
+        <link name="pillar_telescope_link">
+            <visual>
+                <geometry>
+                    <mesh filename="package://poli_description/meshes/components/pillar_telescope.STL" />
                 </geometry>
             </visual>

Commit message: added pillar mounting plate

File: poli_description/robots/poli.urdf.xacro (robot description, xacro)
@@ -107,4 +107,7 @@
             <origin xyz="0.2315586 0 0.0075" rpy="0 -${HALF_PI} 0"/>
         </xacro:pillar>
+        <xacro:pillar_plate parent="pillar_telescope_link">
+            <origin xyz="-0.14899868 0.17604938 -0.14899868" rpy="0 0 0"/>
+        </xacro:pillar_plate>
     </xacro:macro>
 </robot>

Commit message: added additional baseplate threadboard

File: poli_description/robots/poli.urdf.xacro (robot description, xacro)
@@ -30,4 +30,6 @@
     <xacro:include filename="$(find poli_description)/urdf/accessories.urdf.xacro" />
     <xacro:include filename="$(find poli_description)/urdf/poli_components/base_plate.urdf.xacro"/>
+    <xacro:include filename="$(find poli_description)/urdf/poli_components/rmp_plate2.urdf.xacro"/>
+    <xacro:include filename="$(find poli_description)/urdf/poli_components/rmp_plate3.urdf.xacro"/>
     <xacro:include filename="$(find poli_description)/urdf/poli_components/pillar.urdf.xacro"/>
     <xacro:include filename="$(find poli_description)/urdf/poli_components/pillar_plate.urdf.xacro"/>
@@ -104,4 +106,10 @@
             <origin xyz="0.0762 0.16355 0.076" rpy="${HALF_PI} 0 -${HALF_PI}"/>
         </xacro:base_plate>
+        <xacro:rmp_plate2 parent="base_plate_link">
+            <origin xyz="-0.079 0 0.075" rpy="0 0 0"/>
+        </xacro:rmp_plate2>
+        <xacro:rmp_plate3 parent="base_plate_link">
+            <origin xyz="-0.079 0.048 0.075" rpy="${M_PI} 0 0"/>
+        </xacro:rmp_plate3>
         <xacro:pillar parent="base_plate_link">
             <origin xyz="0.2315586 0 0.0075" rpy="0 -${HALF_PI} 0"/>

Commit message: added both lasers. general cleanup of unused sensor descriptions

File: poli_description/robots/poli.urdf.xacro (robot description, xacro)
@@ -28,5 +28,6 @@
     <xacro:include filename="$(find poli_description)/urdf/segway_components/hmi_box_110.urdf.xacro" />
     <xacro:include filename="$(find poli_description)/urdf/segway_components/hmi_plate_110.urdf.xacro" />
-    <xacro:include filename="$(find poli_description)/urdf/accessories.urdf.xacro" />
+    <xacro:include filename="$(find poli_description)/urdf/sensors/hokuyo_ust10lx.urdf.xacro"/>
+    <xacro:include filename="$(find poli_description)/urdf/sensors/hokuyo_ust30lx.urdf.xacro"/>
     <xacro:include filename="$(find poli_description)/urdf/poli_components/base_plate.urdf.xacro"/>
     <xacro:include filename="$(find poli_description)/urdf/poli_components/rmp_plate2.urdf.xacro"/>
@@ -36,4 +37,6 @@
     <property name="M_PI" value="3.14159"/>
     <property name="HALF_PI" value="1.57079"/>
+    <property name="FRONT_LASER_PREFIX" value="front_laser"/>
+    <property name="REAR_LASER_PREFIX" value="rear_laser"/>
     <!-- Wheel Mounting Positions -->
     <xacro:property name="track" value="0.48122440" />
@@ -107,5 +110,5 @@
         </xacro:base_plate>
         <xacro:rmp_plate2 parent="base_plate_link">
-            <origin xyz="-0.079 0 0.075" rpy="0 0 0"/>
+            <origin xyz="-0.079 -0.016 0.075" rpy="0 0 0"/>
         </xacro:rmp_plate2>
         <xacro:rmp_plate3 parent="base_plate_link">
@@ -118,4 +121,11 @@
             <origin xyz="-0.14899868 0.17604938 -0.14899868" rpy="0 0 0"/>
         </xacro:pillar_plate>
+        <!-- Poli Sensors -->
+        <xacro:hokuyo_ust30lx laser_prefix="${FRONT_LASER_PREFIX}" parent="rmp_plate2_link">
+            <origin xyz="0.242 0.075 0.33" rpy="-${HALF_PI} -${HALF_PI} 0" />
+        </xacro:hokuyo_ust30lx>
+        <xacro:hokuyo_ust10lx laser_prefix="${REAR_LASER_PREFIX}" parent="rmp_plate3_link">
+            <origin xyz="0.242 -0.015 0.33" rpy="${HALF_PI} -${HALF_PI} 0" />
+        </xacro:hokuyo_ust10lx>
     </xacro:macro>
 </robot>

Commit message: Merge initial robot description (#11)
* added meshes of basic components. baseplate is added and positioned correctly

* position changes for base plate. added pillar

* flipped baseplate to match reality. added telescope to pillar

* added pillar mounting plate

* added additional baseplate threadboard

* added both lasers. general cleanup of unused sensor descriptions

* removed remaining references to environment configuration #4

File: poli_description/robots/poli.urdf.xacro (robot description, xacro)
@@ -1,5 +1,131 @@
 <?xml version="1.0"?>
+<!--
+Software License Agreement (BSD)
+Copyright (c) 2017, University of Texas Austin
+Author Maxwell Svetlik
+Redistribution and use in source and binary forms, with or without modification, are permitted provided that
+the following conditions are met:
+ * Redistributions of source code must retain the above copyright notice, this list of conditions and the
+   following disclaimer.
+ * Redistributions in binary form must reproduce the above copyright notice, this list of conditions and the
+   following disclaimer in the documentation and/or other materials provided with the distribution.
+ * Neither the name of Stanley Innovation, Inc. nor the names of its contributors may be used to endorse or promote
+   products derived from this software without specific prior written permission.
+THIS SOFTWARE IS PROVIDED BY THE COPYRIGHT HOLDERS AND CONTRIBUTORS "AS IS" AND ANY EXPRESS OR IMPLIED WAR-
+RANTIES, INCLUDING, BUT NOT LIMITED TO, THE IMPLIED WARRANTIES OF MERCHANTABILITY AND FITNESS FOR A PARTICULAR
+PURPOSE ARE DISCLAIMED. IN NO EVENT SHALL THE COPYRIGHT HOLDER OR CONTRIBUTORS BE LIABLE FOR ANY DIRECT, IN-
+DIRECT, INCIDENTAL, SPECIAL, EXEMPLARY, OR CONSEQUENTIAL DAMAGES (INCLUDING, BUT NOT LIMITED TO, PROCUREMENT
+OF SUBSTITUTE GOODS OR SERVICES; LOSS OF USE, DATA, OR PROFITS; OR BUSINESS INTERRUPTION) HOWEVER CAUSED AND
+ON ANY THEORY OF LIABILITY, WHETHER IN CONTRACT, STRICT LIABILITY, OR TORT (INCLUDING NEGLIGENCE OR OTHERWISE)
+ARISING IN ANY WAY OUT OF THE USE OF THIS SOFTWARE, EVEN IF ADVISED OF THE POSSIBILITY OF SUCH DAMAGE.
+-->
 <robot name="segway_robot" xmlns:xacro="http://ros.org/wiki/xacro">
-  <xacro:include filename="$(find poli_description)/urdf/RMP_110/rmp.urdf.xacro" />
-  <xacro:segway_robot />
+    <!-- Included URDF/XACRO Files -->
+    <xacro:include filename="$(find poli_description)/urdf/segway_components/battery.urdf.xacro" />
+    <xacro:include filename="$(find poli_description)/urdf/segway_components/i2_wheel.urdf.xacro" />
+    <xacro:include filename="$(find poli_description)/urdf/segway_components/caster_assembly_110.urdf.xacro" />
+    <xacro:include filename="$(find poli_description)/urdf/segway_components/powerbase_110.urdf.xacro" />
+    <xacro:include filename="$(find poli_description)/urdf/segway_components/hmi_box_110.urdf.xacro" />
+    <xacro:include filename="$(find poli_description)/urdf/segway_components/hmi_plate_110.urdf.xacro" />
+    <xacro:include filename="$(find poli_description)/urdf/sensors/hokuyo_ust10lx.urdf.xacro"/>
+    <xacro:include filename="$(find poli_description)/urdf/sensors/hokuyo_ust30lx.urdf.xacro"/>
+    <xacro:include filename="$(find poli_description)/urdf/poli_components/base_plate.urdf.xacro"/>
+    <xacro:include filename="$(find poli_description)/urdf/poli_components/rmp_plate2.urdf.xacro"/>
+    <xacro:include filename="$(find poli_description)/urdf/poli_components/rmp_plate3.urdf.xacro"/>
+    <xacro:include filename="$(find poli_description)/urdf/poli_components/pillar.urdf.xacro"/>
+    <xacro:include filename="$(find poli_description)/urdf/poli_components/pillar_plate.urdf.xacro"/>
+    <property name="M_PI" value="3.14159"/>
+    <property name="HALF_PI" value="1.57079"/>
+    <property name="FRONT_LASER_PREFIX" value="front_laser"/>
+    <property name="REAR_LASER_PREFIX" value="rear_laser"/>
+    <!-- Wheel Mounting Positions -->
+    <xacro:property name="track" value="0.48122440" />
+    <xacro:property name="wheel_vertical_offset" value="0.08255015" />
+    <!-- Wheel Properties -->
+    <xacro:property name="wheel_length" value="0.09224900" />
+    <xacro:property name="wheel_radius" value="0.2405681" />
+    <xacro:macro name="segway_robot">
+        <gazebo>
+          <plugin name="gazebo_ros_control" filename="libgazebo_ros_control.so">
+              <robotNamespace>/</robotNamespace>
+          </plugin>
+        </gazebo>
+        <!-- Base link is the center of the robot's chassis between the motors projected on the ground -->
+        <link name="base_link"/>
+        <!--Chassis -->
+        <xacro:powerbase_110 chassis_prefix="base" parent="base_link">
+            <origin xyz="0 0 ${-wheel_vertical_offset + wheel_radius}" rpy="0 0 0" />
+        </xacro:powerbase_110>
+        <link name="inertial_collision_link">
+			<inertial>
+				<mass value="29.756375" />
+				<origin xyz="0.001751 0.000008 0.018544" />
+				<inertia ixx="0.696269"  ixy="0.016133" ixz="0.003232"
+                         iyx="0.016133"  iyy="0.299110" iyz="-0.000004"
+                         izx="-0.077476" izy="-0.000004" izz="0.864394" />
+			</inertial>
+            <collision>
+				<geometry>
+					<mesh filename="package://poli_description/meshes/collision/110_powerbase_collision.stl" />
+				</geometry>
+			</collision>
+		</link>
+		<joint name="inertial_collision_joint" type="fixed" >
+		    <parent link="base_chassis_link" />
+		    <child link="inertial_collision_link" />
+		</joint>
+        <!-- Propulsion Batteries -->
+        <xacro:battery battery_prefix="mcu_1" parent="base_chassis_link">
+            <origin xyz="-0.09298 0 0" rpy="0 0 0" />
+        </xacro:battery>
+        <!-- Aux Batteries -->
+        <xacro:battery battery_prefix="aux" parent="base_chassis_link">
+            <origin xyz="0.09298 0 0" rpy="0 0 ${M_PI}" />
+        </xacro:battery>
+        <!-- HMI Box -->
+        <xacro:hmi_box_110 parent="base_chassis_link">
+            <origin xyz="0 0 0.09504494" rpy="0 0 0" />
+        </xacro:hmi_box_110>
+        <xacro:hmi_plate_110 parent="hmi_link">
+            <origin xyz="0 0 0" rpy="0 0 0" />
+        </xacro:hmi_plate_110>
+        <!-- Segway wheel macros -->
+        <xacro:i2_wheel wheel_prefix="left" parent="base_chassis_link" visual_rotation="0.0">
+            <origin xyz="0 ${track/2} ${wheel_vertical_offset}" rpy="0 0 0" />
+        </xacro:i2_wheel>
+        <xacro:i2_wheel wheel_prefix="right" parent="base_chassis_link" visual_rotation="${M_PI}">
+            <origin xyz="0 ${-track/2} ${wheel_vertical_offset}" rpy="0 0 0" />
+        </xacro:i2_wheel>
+        <!-- Segway Caster Assembly-->
+        <xacro:caster_assembly_110 caster_prefix="rear" parent="base_chassis_link">
+            <origin xyz="-0.32784550 0 0.03326933" rpy="0 0 ${M_PI}" />
+        </xacro:caster_assembly_110>
+        <xacro:caster_assembly_110 caster_prefix="front" parent="base_chassis_link">
+            <origin xyz="0.32784550 0 0.03326933" rpy="0 0 0" />
+        </xacro:caster_assembly_110>
+        <!-- Setup any accessories defined in the environment -->
+        <xacro:segway_accessories />
+        <xacro:base_plate parent="base_chassis_link">
+            <origin xyz="0.0762 0.16355 0.076" rpy="${HALF_PI} 0 -${HALF_PI}"/>
+        </xacro:base_plate>
+        <xacro:rmp_plate2 parent="base_plate_link">
+            <origin xyz="-0.079 -0.016 0.075" rpy="0 0 0"/>
+        </xacro:rmp_plate2>
+        <xacro:rmp_plate3 parent="base_plate_link">
+            <origin xyz="-0.079 0.048 0.075" rpy="${M_PI} 0 0"/>
+        </xacro:rmp_plate3>
+        <xacro:pillar parent="base_plate_link">
+            <origin xyz="0.2315586 0 0.0075" rpy="0 -${HALF_PI} 0"/>
+        </xacro:pillar>
+        <xacro:pillar_plate parent="pillar_telescope_link">
+            <origin xyz="-0.14899868 0.17604938 -0.14899868" rpy="0 0 0"/>
+        </xacro:pillar_plate>
+        <!-- Poli Sensors -->
+        <xacro:hokuyo_ust30lx laser_prefix="${FRONT_LASER_PREFIX}" parent="rmp_plate2_link">
+            <origin xyz="0.242 0.075 0.33" rpy="-${HALF_PI} -${HALF_PI} 0" />
+        </xacro:hokuyo_ust30lx>
+        <xacro:hokuyo_ust10lx laser_prefix="${REAR_LASER_PREFIX}" parent="rmp_plate3_link">
+            <origin xyz="0.242 -0.015 0.33" rpy="${HALF_PI} -${HALF_PI} 0" />
+        </xacro:hokuyo_ust10lx>
+    </xacro:macro>
 </robot>
