Commit message: modified STL origin allowing perfect alignment

File: poli_description/robots/jaco2_custom.xacro (robot description, xacro)
@@ -17,4 +17,5 @@
     <xacro:include filename="$(find kinova_description)/urdf/kinova_finger_set.xacro" />
     <xacro:include filename="$(find poli_description)/urdf/poli_components/weiss_mount.urdf.xacro"/>
+    <xacro:include filename="$(find wsg_50_simulation)/urdf/wsg_50.urdf.xacro"/>
     <!-- Import all Gazebo-customization elements -->
     <xacro:include filename="$(find kinova_description)/urdf/kinova.gazebo" />
@@ -117,7 +118,10 @@
         <xacro:kinova_armjoint joint_name="${prefix}_joint_6" type="${joint_6_type}" parent="${prefix}_link_5" child="${prefix}_link_6" joint_axis_xyz="${joint_6_axis_xyz}" joint_origin_xyz="${joint_6_origin_xyz}" joint_origin_rpy="${joint_6_origin_rpy}" joint_lower_limit="${joint_6_lower_limit}" joint_upper_limit="${joint_6_upper_limit}"/>
         <xacro:weiss_mount link_name="${prefix}_link_7" parent="${prefix}_link_6">
+            <origin xyz="${joint_7_origin_xyz}" rpy="-${J_PI/2} 0 0"/>
+        </xacro:weiss_mount>
+        <xacro:wsg_50_xacro name="gripper" parent="${prefix}_link_7">
             <origin xyz="0 0 0" rpy="0 0 0"/>
-        </xacro:weiss_mount>
-       <xacro:kinova_armjoint joint_name="${prefix}_joint_7" type="${joint_7_type}" parent="${prefix}_link_6" child="${prefix}_link_7" joint_axis_xyz="${joint_7_axis_xyz}" joint_origin_xyz="${joint_7_origin_xyz}" joint_origin_rpy="${joint_7_origin_rpy}" joint_lower_limit="${joint_7_lower_limit}" joint_upper_limit="${joint_7_upper_limit}"/>
+        </xacro:wsg_50_xacro>
+        <xacro:kinova_armjoint joint_name="${prefix}_joint_7" type="${joint_7_type}" parent="${prefix}_link_6" child="${prefix}_link_7" joint_axis_xyz="${joint_7_axis_xyz}" joint_origin_xyz="${joint_7_origin_xyz}" joint_origin_rpy="${joint_7_origin_rpy}" joint_lower_limit="${joint_7_lower_limit}" joint_upper_limit="${joint_7_upper_limit}"/>
         <!--
         <xacro:kinova_virtual_link link_name="${prefix}_end_effector"/>

File: poli_description/urdf/poli_components/weiss_mount.urdf.xacro (robot description, xacro)
@@ -22,5 +22,4 @@
 <robot xmlns:xacro="http://ros.org/wiki/xacro" name="weiss_mount">
     <xacro:macro name="weiss_mount" params="parent link_name *origin">
-        <!--
         <joint name="weiss_mount_joint" type="fixed">
             <xacro:insert_block name="origin" />
@@ -28,5 +27,4 @@
             <child link="${link_name}" />
         </joint>
-        -->
         <link name="${link_name}">
             <visual>

Commit message: added wsg 32 gripper

File: poli_description/robots/jaco2_custom.xacro (robot description, xacro)
@@ -17,5 +17,5 @@
     <xacro:include filename="$(find kinova_description)/urdf/kinova_finger_set.xacro" />
     <xacro:include filename="$(find poli_description)/urdf/poli_components/weiss_mount.urdf.xacro"/>
-    <xacro:include filename="$(find wsg_50_simulation)/urdf/wsg_50.urdf.xacro"/>
+    <xacro:include filename="$(find wsg_32_description)/robots/wsg_32_description.urdf.xacro"/>
     <!-- Import all Gazebo-customization elements -->
     <xacro:include filename="$(find kinova_description)/urdf/kinova.gazebo" />
@@ -120,8 +120,10 @@
             <origin xyz="${joint_7_origin_xyz}" rpy="-${J_PI/2} 0 0"/>
         </xacro:weiss_mount>
-        <xacro:wsg_50_xacro name="gripper" parent="${prefix}_link_7">
-            <origin xyz="0 0 0" rpy="0 0 0"/>
-        </xacro:wsg_50_xacro>
+        <xacro:wsg_32_xacro name="gripper" parent="${prefix}_link_7">
+            <origin xyz="0.0001 0 0.085" rpy="0 0 -${J_PI/2}"/>
+        </xacro:wsg_32_xacro>
+        <!--
         <xacro:kinova_armjoint joint_name="${prefix}_joint_7" type="${joint_7_type}" parent="${prefix}_link_6" child="${prefix}_link_7" joint_axis_xyz="${joint_7_axis_xyz}" joint_origin_xyz="${joint_7_origin_xyz}" joint_origin_rpy="${joint_7_origin_rpy}" joint_lower_limit="${joint_7_lower_limit}" joint_upper_limit="${joint_7_upper_limit}"/>
+        -->
         <!--
         <xacro:kinova_virtual_link link_name="${prefix}_end_effector"/>

Commit message: made adjustments to run gripper and arm as a live system. note that to run the kinova arm launch file, the kinova_robot.launch file must not run any nodes under its urdf flag

File: poli_description/robots/jaco2_custom.xacro (robot description, xacro)
@@ -117,8 +117,8 @@
         <xacro:kinova_armlink link_name="${prefix}_link_6" link_mesh="${link_6_mesh}" use_ring_mesh="true" ring_mesh="ring_small" mesh_no="${link_6_mesh_no}"/>
         <xacro:kinova_armjoint joint_name="${prefix}_joint_6" type="${joint_6_type}" parent="${prefix}_link_5" child="${prefix}_link_6" joint_axis_xyz="${joint_6_axis_xyz}" joint_origin_xyz="${joint_6_origin_xyz}" joint_origin_rpy="${joint_6_origin_rpy}" joint_lower_limit="${joint_6_lower_limit}" joint_upper_limit="${joint_6_upper_limit}"/>
-        <xacro:weiss_mount link_name="${prefix}_link_7" parent="${prefix}_link_6">
+        <xacro:weiss_mount link_name="${prefix}_link_7" joint_name="${prefix}_joint_7" parent="${prefix}_link_6">
             <origin xyz="${joint_7_origin_xyz}" rpy="-${J_PI/2} 0 0"/>
         </xacro:weiss_mount>
-        <xacro:wsg_32_xacro name="gripper" parent="${prefix}_link_7">
+        <xacro:wsg_32_xacro name="wsg_50_gripper" parent="${prefix}_link_7">
             <origin xyz="0.0001 0 0.085" rpy="0 0 -${J_PI/2}"/>
         </xacro:wsg_32_xacro>

File: poli_description/urdf/poli_components/weiss_mount.urdf.xacro (robot description, xacro)
@@ -21,6 +21,6 @@
 -->
 <robot xmlns:xacro="http://ros.org/wiki/xacro" name="weiss_mount">
-    <xacro:macro name="weiss_mount" params="parent link_name *origin">
-        <joint name="weiss_mount_joint" type="continuous">
+    <xacro:macro name="weiss_mount" params="parent joint_name link_name *origin">
+        <joint name="${joint_name}" type="continuous">
             <xacro:insert_block name="origin" />
             <parent link="${parent}" />
