Commit message: modified wrist to be continuous rather than fixed

File: poli_description/urdf/poli_components/weiss_mount.urdf.xacro (robot description, xacro)
@@ -22,8 +22,10 @@
 <robot xmlns:xacro="http://ros.org/wiki/xacro" name="weiss_mount">
     <xacro:macro name="weiss_mount" params="parent link_name *origin">
-        <joint name="weiss_mount_joint" type="fixed">
+        <joint name="weiss_mount_joint" type="continuous">
             <xacro:insert_block name="origin" />
             <parent link="${parent}" />
             <child link="${link_name}" />
+            <axis xyz="0 0 1"/>
+            <limit effort="50" velocity="50"/>
         </joint>
         <link name="${link_name}">
