Commit message: along with last commit, enables pillar to be in overall robot state

File: poli2_description/urdf/poli_components/pillar.urdf.xacro (robot description, xacro)
@@ -39,5 +39,5 @@
             </collision>
         </link>
-        <joint name="pillar_telescope_joint" type="fixed">
+        <joint name="pillar_telescope_joint" type="prismatic">
             <origin xyz="0.2175586 0.1 0.02" rpy="0 -1.570796 0"/>
             <parent link="${parent}" />
