Commit message: corrected joint limits for assumed starting position for tilt

File: poli2_description/urdf/poli_components/neck_mount.urdf.xacro (robot description, xacro)
@@ -162,5 +162,6 @@
   <joint
     name="tilt_joint"
-    type="continuous">
+    type="revolute">
+    <limit lower="-0.7" upper="0.8" velocity="1.0" effort="1.0"/>
     <origin
       xyz="0.1011 0 -0.00960000000000004"

Commit message: fixed urdf to have less warnings and added in some basic controllers to move the head and arm. controllers are not yet tested

File: poli2_description/urdf/poli_components/neck_mount.urdf.xacro (robot description, xacro)
@@ -184,4 +184,14 @@
     </actuator>
   </transmission>
+  <transmission name="pan_joint_trans">
+    <type>transmission_interface/SimpleTransmission</type>
+    <joint name="pan_joint">
+      <hardwareInterface>hardware_interface/PositionJointInterface</hardwareInterface>
+    </joint>
+    <actuator name="pan_joint_actuator">
+	 <!--mechanicalReduction>29768</mechanicalReduction-->
+	 <mechanicalReduction>160</mechanicalReduction>
+    </actuator>
+  </transmission>
   </xacro:macro>
 </robot>

File: poli2_description/urdf/segway_components/caster_assembly_110.urdf.xacro (robot description, xacro)
@@ -87,8 +87,8 @@
 			<type>transmission_interface/SimpleTransmission</type>
 			<joint name="${caster_prefix}_caster_swivel">
-			    <hardwareInterface>EffortJointInterface</hardwareInterface>
+			    <hardwareInterface>hardware_interface/EffortJointInterface</hardwareInterface>
 			</joint>
 			<actuator name="${caster_prefix}_caster_swivel_motor">
-			    <hardwareInterface>EffortJointInterface</hardwareInterface>
+			    <hardwareInterface>hardware_interface/EffortJointInterface</hardwareInterface>
 				<mechanicalReduction>1</mechanicalReduction>
 			</actuator>
@@ -134,8 +134,8 @@
 			<type>transmission_interface/SimpleTransmission</type>
 			<joint name="${caster_prefix}_caster_wheel">
-			    <hardwareInterface>EffortJointInterface</hardwareInterface>
+			    <hardwareInterface>hardware_interface/EffortJointInterface</hardwareInterface>
 			</joint>
 			<actuator name="${caster_prefix}_caster_wheel_motor">
-			    <hardwareInterface>EffortJointInterface</hardwareInterface>
+			    <hardwareInterface>hardware_interface/EffortJointInterface</hardwareInterface>
 				<mechanicalReduction>1</mechanicalReduction>
 			</actuator>

File: poli2_description/urdf/segway_components/i2_wheel.urdf.xacro (robot description, xacro)
@@ -64,5 +64,5 @@
 			</actuator>
 			<joint name="${wheel_prefix}_wheel">
-				<hardwareInterface>VelocityJointInterface</hardwareInterface>
+				<hardwareInterface>hardware_interface/VelocityJointInterface</hardwareInterface>
 			</joint>
 		</transmission>

File: poli2_description/urdf/segway_components/x2_wheel.urdf.xacro (robot description, xacro)
@@ -64,5 +64,5 @@
 			</actuator>
 			<joint name="${wheel_prefix}_wheel">
-				<hardwareInterface>VelocityJointInterface</hardwareInterface>
+				<hardwareInterface>hardware_interface/VelocityJointInterface</hardwareInterface>
 			</joint>
 		</transmission>
