Commit message: fixed standalone description files for jaco2 custom

File: poli2_description/robots/jaco2_custom_wrapper.urdf (robot description, URDF)
Before this commit: robot j2s7s300, 15 links, 14 joints
Links:
- link j2s7s300_link_7: geometry collision mesh filename=package://poli2_description/meshes/components/weiss_mount.S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; visual mesh filename=package://poli2_description/meshes/components/weiss_mount.S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
Joints:
- joint j2s7s300_joint_7: axis 0 0 1 -> 0 0 -1

File: poli2_description/robots/jaco2_custom_wrapper.xacro (robot description, xacro)
@@ -38,4 +38,4 @@
   </joint>
   <property name="robot_root" value="root" />
-  <xacro:jaco2_custom  base_parent="${robot_root}"/>
+  <xacro:jaco2_custom  base_parent="${robot_root}"  base_origin_xyz="0 0 0" base_origin_rpy="0 0 0"/>
 </robot>
