Commit message: modified collision geometries to be accurate according to mesh model. fixed wrist rotational issue wrt the model vs reality.

File: poli2_description/robots/poli.urdf (robot description, URDF)
Before this commit: robot segway_robot, 36 links, 35 joints
Links:
- link base_plate_link: geometry collision mesh filename=package://poli2_description/meshes/components/base_plate.STL; visual mesh filename=package://poli2_description/meshes/components/base_plate.STL
- link front_laser_link: geometry collision mesh filename=package://poli2_description/meshes/visual/sensors/hokuyo_us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; visual mesh filename=package://poli2_description/meshes/visual/sensors/hokuyo_us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
- link j2s7s300_link_7: geometry collision mesh filename=package://poli2_description/meshes/components/weiss_mount.S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; visual mesh filename=package://poli2_description/meshes/components/weiss_mount.S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
- link pillar_base_link: geometry collision mesh filename=package://poli2_description/meshes/components/pillar_exteri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; visual mesh filename=package://poli2_description/meshes/components/pillar_exteri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
- link pillar_plate_link: geometry collision mesh filename=package://poli2_description/meshes/components/pillar_plate.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; visual mesh filename=package://poli2_description/meshes/components/pillar_plate.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
- link pillar_telescope_link: geometry collision mesh filename=package://poli2_description/meshes/components/pillar_telesc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; visual mesh filename=package://poli2_description/meshes/components/pillar_telesc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
- link rear_laser_link: geometry collision mesh filename=package://poli2_description/meshes/visual/sensors/hokuyo_us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; visual mesh filename=package://poli2_description/meshes/visual/sensors/hokuyo_us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
- link rmp_plate2_link: geometry collision mesh filename=package://poli2_description/meshes/components/rmp_plate2.STL; visual mesh filename=package://poli2_description/meshes/components/rmp_plate2.STL
- link rmp_plate3_link: geometry collision mesh filename=package://poli2_description/meshes/components/rmp_plate3.STL; visual mesh filename=package://poli2_description/meshes/components/rmp_plate3.STL
Joints:
- joint j2s7s300_joint_7: axis 0 0 1 -> 0 0 -1

File: poli2_description/urdf/poli_components/base_plate.urdf.xacro (robot description, xacro)
@@ -35,5 +35,5 @@
             <collision>
                 <geometry>
-                    <box size="0.1 0.1 0.1"/>
+                    <mesh filename="package://poli2_description/meshes/components/base_plate.STL" />
                 </geometry>
             </collision>

File: poli2_description/urdf/poli_components/pillar.urdf.xacro (robot description, xacro)
@@ -35,5 +35,5 @@
             <collision>
                 <geometry>
-                    <box size="0.1 0.1 0.1"/>
+                    <mesh filename="package://poli2_description/meshes/components/pillar_exterior.STL" />
                 </geometry>
             </collision>
@@ -54,5 +54,5 @@
             <collision>
                 <geometry>
-                    <box size="0.1 0.1 0.1"/>
+                    <mesh filename="package://poli2_description/meshes/components/pillar_telescope.STL" />
                 </geometry>
             </collision>

File: poli2_description/urdf/poli_components/pillar_plate.urdf.xacro (robot description, xacro)
@@ -35,5 +35,5 @@
             <collision>
                 <geometry>
-                    <box size="0.1 0.1 0.1"/>
+                    <mesh filename="package://poli2_description/meshes/components/pillar_plate.STL" />
                 </geometry>
             </collision>

File: poli2_description/urdf/poli_components/rmp_plate2.urdf.xacro (robot description, xacro)
@@ -35,5 +35,5 @@
             <collision>
                 <geometry>
-                    <box size="0.1 0.1 0.1"/>
+                    <mesh filename="package://poli2_description/meshes/components/rmp_plate2.STL" />
                 </geometry>
             </collision>

File: poli2_description/urdf/poli_components/rmp_plate3.urdf.xacro (robot description, xacro)
@@ -35,5 +35,5 @@
             <collision>
                 <geometry>
-                    <box size="0.1 0.1 0.1"/>
+                    <mesh filename="package://poli2_description/meshes/components/rmp_plate3.STL" />
                 </geometry>
             </collision>

File: poli2_description/urdf/poli_components/weiss_mount.urdf.xacro (robot description, xacro)
@@ -26,5 +26,5 @@
             <parent link="${parent}" />
             <child link="${link_name}" />
-            <axis xyz="0 0 1"/>
+            <axis xyz="0 0 -1"/>
             <limit effort="50" velocity="50"/>
         </joint>
@@ -37,5 +37,5 @@
             <collision>
                 <geometry>
-                    <box size="0.1 0.1 0.1"/>
+                    <mesh filename="package://poli2_description/meshes/components/weiss_mount.STL" />
                 </geometry>
             </collision>

File: poli2_description/urdf/sensors/hokuyo_ust10lx.urdf.xacro (robot description, xacro)
@@ -36,5 +36,5 @@
             <collision>
                 <geometry>
-                    <box size="0.1 0.1 0.1"/>
+                    <mesh filename="package://poli2_description/meshes/visual/sensors/hokuyo_ustlx.dae" />
                 </geometry>
             </collision>

File: poli2_description/urdf/sensors/hokuyo_ust30lx.urdf.xacro (robot description, xacro)
@@ -36,5 +36,5 @@
             <collision>
                 <geometry>
-                    <box size="0.1 0.1 0.1"/>
+                    <mesh filename="package://poli2_description/meshes/visual/sensors/hokuyo_ustlx.dae" />
                 </geometry>
             </collision>

Commit message: regenerated urdf with changes in wsg_32_description. accurately shows finger movement

File: poli2_description/robots/poli.urdf (robot description, URDF)
Before this commit: robot segway_robot, 36 links, 35 joints
Joints:
- joint wsg_50_gripper_base_joint_gripper_left: axis 0 1 0 -> 0 -1 0; origin xyz=-0.0003903 -0.0358 0.069014 rpy=3.1416 -1.5708 0 -> xyz=-0.0003903 -0.0078 0.069014 rpy=3.1416 -1.5708 0
- joint wsg_50_gripper_base_joint_gripper_right: axis 0 0 -1 -> 0 0 1; limit lower=-0.028 upper=0 effort=0 velocity=0 -> lower=0 upper=0.028 effort=0 velocity=0; origin xyz=-0.0003903 0.0358 0.069012 rpy=1.5708 -1.5708 0 -> xyz=-0.0003903 0.0078 0.069012 rpy=-1.5708 -1.5708 0
- joint wsg_50_gripper_right_universal_finger_joint: origin xyz=0.00755 0.0 0.0049 rpy=0 1.57079 -1.57079 -> xyz=0.00755 0.0 0.0049 rpy=0 -1.57079 -1.57079

Commit message: fixed joint limits for pan; joint state mapping; regenerated moveit config with pan_tilt

File: poli2_description/robots/poli.urdf (robot description, URDF)
Before this commit: robot segway_robot, 36 links, 35 joints
Links:
- added link neck_base_link, mass 0.557568366166049; collision mesh filename=package://poli2_description/meshes/components/neck/base_lin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; visual mesh filename=package://poli2_description/meshes/components/neck/base_lin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
- added link pan_link, mass 0.661811908284221; collision mesh filename=package://poli2_description/meshes/components/neck/pan_link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; visual mesh filename=package://poli2_description/meshes/components/neck/pan_link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
- added link tilt_link, mass 0.0557850572590686; collision mesh filename=package://poli2_description/meshes/components/neck/tilt_lin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; visual mesh filename=package://poli2_description/meshes/components/neck/tilt_lin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
Joints:
- added joint neck_base_joint: type fixed, parent pillar_plate_link, child neck_base_link, origin xyz=0.22 0.385 0.19 rpy=0 0 1.57079, limit effort=50 velocity=50
- added joint pan_joint: type revolute, parent neck_base_link, child pan_link, origin xyz=0.0179 0 0 rpy=0 0 0, axis 1 0 0, limit lower=-1.54 upper=1.54 effort=30 velocity=1.0
- added joint tilt_joint: type revolute, parent pan_link, child tilt_link, origin xyz=0.1011 0 -0.00960000000000004 rpy=-1.5707963267949 0 -1.5707963267949, axis 0 1 0, limit lower=-0.7 upper=0.8 effort=1.0 velocity=1.0

File: poli2_description/urdf/poli_components/neck_mount.urdf.xacro (robot description, xacro)
@@ -109,5 +109,6 @@
   <joint
     name="pan_joint"
-    type="continuous">
+    type="revolute">
+    <limit lower="-1.54" upper="1.54" velocity="1.0" effort="30"/>
     <origin
       xyz="0.0179 0 0"

Commit message: fixed urdf to match reality wrt the arm

File: poli2_description/robots/poli.urdf (robot description, URDF)
Before this commit: robot segway_robot, 39 links, 38 joints
Links:
- added link camera_depth_frame
- added link camera_depth_optical_frame
- added link camera_link, mass 0.564; collision box size=0.0400 0.1650 0.0300; visual mesh filename=package://poli2_description/meshes/sensors/astra.dae scale=1 1 1
- added link camera_rgb_frame
- added link camera_rgb_optical_frame
Joints:
- added joint camera_depth_joint: type fixed, parent camera_rgb_frame, child camera_depth_frame, origin xyz=0 0.025 0 rpy=0 0 0
- added joint camera_depth_optical_joint: type fixed, parent camera_depth_frame, child camera_depth_optical_frame, origin xyz=0 0 0 rpy=-1.570795 0 -1.570795
- added joint camera_joint: type fixed, parent camera_rgb_frame, child camera_link, origin xyz=0 -0.0125 0 rpy=0 0 0
- added joint camera_rgb_joint: type fixed, parent tilt_link, child camera_rgb_frame, origin xyz=-0.08 -0.0035 0.05 rpy=0 0 3.14159
- added joint camera_rgb_optical_joint: type fixed, parent camera_rgb_frame, child camera_rgb_optical_frame, origin xyz=0 0 0 rpy=-1.570795 0 -1.570795
- joint j2s7s300_joint_base: origin xyz=0 0 0 rpy=-1.57079 -1.57079 0 -> xyz=0 0.05 0.0575 rpy=-1.57079 -1.57079 0
- joint neck_base_joint: origin xyz=0.22 0.385 0.19 rpy=0 0 1.57079 -> xyz=0.1785 0.385 0.205 rpy=0 0 1.57079

File: poli2_description/robots/poli.urdf.xacro (robot description, xacro)
@@ -30,4 +30,5 @@
     <xacro:include filename="$(find poli2_description)/urdf/sensors/hokuyo_ust10lx.urdf.xacro"/>
     <xacro:include filename="$(find poli2_description)/urdf/sensors/hokuyo_ust30lx.urdf.xacro"/>
+    <xacro:include filename="$(find poli2_description)/urdf/sensors/astra.urdf.xacro"/>
     <xacro:include filename="$(find poli2_description)/urdf/poli_components/base_plate.urdf.xacro"/>
     <xacro:include filename="$(find poli2_description)/urdf/poli_components/rmp_plate2.urdf.xacro"/>
@@ -133,7 +134,7 @@
         </xacro:pillar_plate>
         <xacro:neck_mount parent="pillar_plate_link">
-            <origin xyz="0.22 0.385 0.19" rpy="0 0 ${HALF_PI}"/>
+            <origin xyz="0.1785 0.385 0.205" rpy="0 0 ${HALF_PI}"/>
         </xacro:neck_mount>
-	<xacro:jaco2_custom base_parent="pillar_plate_link" base_origin_xyz="0 0 0" base_origin_rpy="-${HALF_PI} -${HALF_PI} 0">
+	<xacro:jaco2_custom base_parent="pillar_plate_link" base_origin_xyz="0 0.05 0.0575" base_origin_rpy="-${HALF_PI} -${HALF_PI} 0">
 	</xacro:jaco2_custom>
         <!-- Poli Sensors -->
@@ -144,4 +145,7 @@
             <origin xyz="0.242 -0.015 0.33" rpy="${HALF_PI} -${HALF_PI} 0" />
         </xacro:hokuyo_ust10lx>
+        <xacro:sensor_astra parent="tilt_link">
+	    <origin xyz="-0.08 -0.0035 0.05" rpy="0 0 ${M_PI}"/>
+        </xacro:sensor_astra>
     </xacro:macro>
 </robot>

Commit message: changed model axis of rotation to match actuator

File: poli2_description/robots/poli.urdf (robot description, URDF)
Before this commit: robot segway_robot, 44 links, 43 joints
Joints:
- joint tilt_joint: axis 0 1 0 -> 0 -1 0

File: poli2_description/urdf/poli_components/neck_mount.urdf.xacro (robot description, xacro)
@@ -173,5 +173,5 @@
       link="tilt_link" />
     <axis
-      xyz="0 1 0" />
+      xyz="0 -1 0" />
   </joint>
   <transmission name="tilt_joint_trans">

Commit message: tf and navigation tweaks

File: poli2_description/robots/poli.urdf (robot description, URDF)
Before this commit: robot segway_robot, 44 links, 43 joints
Links:
- added link sonar_link_1, mass 0.564; collision mesh filename=package://poli2_description/meshes/components/sonar_mount_1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; visual mesh filename=package://poli2_description/meshes/components/sonar_mount_1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
Joints:
- added joint sonar_joint: type fixed, parent pillar_plate_link, child sonar_link_1, origin xyz=0.007 0.022 0.203 rpy=1.57079 0 3.14158

File: poli2_description/robots/poli.urdf.xacro (robot description, xacro)
@@ -150,5 +150,5 @@
         </xacro:sensor_astra>
         <xacro:sensor_sonar parent="pillar_plate_link">
-            <origin xyz="0.007 0.022 0.203" rpy="${HALF_PI} 0 ${HALF_PI}"/>
+            <origin xyz="0.007 0.022 0.203" rpy="${HALF_PI} 0 ${HALF_PI*2}"/>
         </xacro:sensor_sonar>
     </xacro:macro>

File: poli2_description/urdf/sensors/sonar.urdf.xacro (robot description, xacro)
@@ -22,5 +22,5 @@
       <inertial>
         <mass value="0.564" />
-        <origin xyz="0 0 0" />
+        <origin xyz="0 0 0"/>
         <inertia ixx="0.003881243" ixy="0.0" ixz="0.0"
                  iyy="0.000498940" iyz="0.0"
@@ -29,5 +29,5 @@
     </link>
     <!-- simulation info -->
-    <gazebo reference="sonar_link">
+    <gazebo reference="sonar_link_1">
       <sensor type="ray" name="sonar">
         <always_on>true</always_on>
