Commit message: initial commit for poli2 simulator stack. still lots of pieces missing

File: poli2_description/robots/jaco2_custom_wrapper.xacro (robot description, xacro)
@@ -37,5 +37,5 @@
     <origin xyz="0 0 0" rpy="0 0 0" />
   </joint>
-  <property name="robot_root" value="root" />
+  <xacro:property name="robot_root" value="root" />
   <xacro:jaco2_custom  base_parent="${robot_root}"  base_origin_xyz="0 0 0" base_origin_rpy="0 0 0"/>
 </robot>

File: poli2_description/urdf/RMP_110/rmp.urdf.xacro (robot description, xacro)
@@ -30,5 +30,5 @@
     <xacro:include filename="$(find poli2_description)/urdf/segway_components/hmi_plate_110.urdf.xacro" />
     <xacro:include filename="$(find poli2_description)/urdf/accessories.urdf.xacro" />
-    <property name="M_PI" value="3.14159"/>
+    <xacro:property name="M_PI" value="3.14159"/>
     <!-- Wheel Mounting Positions -->
     <xacro:property name="track" value="0.48122440" />

File: poli2_description/urdf/poli_components/base_plate.urdf.xacro (robot description, xacro)
@@ -28,4 +28,12 @@
         </joint>
         <link name="base_plate_link">
+			<!-- THESE ARE MADE UP. TODO: REPLACE WITH REAL NUMBERS-->
+            <inertial>
+                <mass value="0.078971" />
+                <origin xyz="-0.000022 -0.000090 0.035623" />
+                <inertia  ixx="0.000082"  ixy="0.000000" ixz="0.000000"
+                          iyx="0.000000" iyy="0.000081"  iyz="-0.000001"
+                          izx="0.000000"  izy="-0.000001" izz="0.000103" />
+            </inertial>
             <visual>
                 <geometry>
