Commit message: residual changes from merge and rename of package

File: poli2_description/robots/jaco2_custom.xacro (robot description, xacro)
@@ -16,5 +16,5 @@
     <xacro:include filename="$(find kinova_description)/urdf/kinova_common.xacro" />
     <xacro:include filename="$(find kinova_description)/urdf/kinova_finger_set.xacro" />
-    <xacro:include filename="$(find poli_description)/urdf/poli_components/weiss_mount.urdf.xacro"/>
+    <xacro:include filename="$(find poli2_description)/urdf/poli_components/weiss_mount.urdf.xacro"/>
     <xacro:include filename="$(find wsg_32_description)/robots/wsg_32_description.urdf.xacro"/>
     <!-- Import all Gazebo-customization elements -->

File: poli2_description/robots/jaco2_custom_wrapper.xacro (robot description, xacro)
@@ -14,5 +14,5 @@
     xmlns:physics="http://playerstage.sourceforge.net/gazebo/xmlschema/#physics"
     xmlns:xacro="http://ros.org/wiki/xacro" name="j2s7s300">
-  <xacro:include filename="$(find poli_description)/robots/jaco2_custom.xacro"/>
+  <xacro:include filename="$(find poli2_description)/robots/jaco2_custom.xacro"/>
   <link name="root">
     <visual>

File: poli2_description/urdf/poli_components/weiss_mount.urdf.xacro (robot description, xacro)
@@ -32,5 +32,5 @@
             <visual>
                 <geometry>
-                    <mesh filename="package://poli_description/meshes/components/weiss_mount.STL" />
+                    <mesh filename="package://poli2_description/meshes/components/weiss_mount.STL" />
                 </geometry>
             </visual>

Commit message: halfway adding jaco to robot

File: poli2_description/robots/jaco2_custom.xacro (robot description, xacro)
@@ -101,8 +101,8 @@
     <property name="joint_end_effector_origin_xyz" value="0 0 -0.1600" />
     <property name="joint_end_effector_origin_rpy" value="${J_PI} 0 0" />
-    <xacro:macro name="jaco2_custom" params="base_parent prefix:=j2s7s300">
+    <xacro:macro name="jaco2_custom" params="base_origin_parent base_xyz base_origin_rpy prefix:=j2s7s300">
         <xacro:gazebo_config robot_namespace="${prefix}"/>
         <xacro:kinova_armlink link_name="${prefix}_link_base" link_mesh="${link_base_mesh}" mesh_no="${link_base_mesh_no}"/>
-        <xacro:kinova_armjoint joint_name="${prefix}_joint_base" type="${joint_base_type}" parent="${base_parent}" child="${prefix}_link_base" joint_axis_xyz="${joint_base_axis_xyz}" joint_origin_xyz="${joint_base_origin_xyz}" joint_origin_rpy="${joint_base_origin_rpy}" joint_lower_limit="0" joint_upper_limit="0" fixed="true"/>
+        <xacro:kinova_armjoint joint_name="${prefix}_joint_base" type="${joint_base_type}" parent="${base_parent}" child="${prefix}_link_base" joint_axis_xyz="${joint_base_axis_xyz}" joint_origin_xyz="${base_origin_xyz}" joint_origin_rpy="${base_origin_rpy}" joint_lower_limit="0" joint_upper_limit="0" fixed="true"/>
         <xacro:kinova_armlink link_name="${prefix}_link_1" link_mesh="${link_1_mesh}" use_ring_mesh="true" mesh_no="${link_1_mesh_no}"/>
         <xacro:kinova_armjoint joint_name="${prefix}_joint_1" type="${joint_1_type}" parent="${prefix}_link_base" child="${prefix}_link_1" joint_axis_xyz="${joint_1_axis_xyz}" joint_origin_xyz="${joint_1_origin_xyz}" joint_origin_rpy="${joint_1_origin_rpy}" joint_lower_limit="${joint_1_lower_limit}" joint_upper_limit="${joint_1_upper_limit}"/>

File: poli2_description/robots/poli.urdf.xacro (robot description, xacro)
@@ -35,4 +35,5 @@
     <xacro:include filename="$(find poli2_description)/urdf/poli_components/pillar.urdf.xacro"/>
     <xacro:include filename="$(find poli2_description)/urdf/poli_components/pillar_plate.urdf.xacro"/>
+    <xacro:include filename="$(find poli2_description)/robots/jaco2_custom.xacro"/>
     <property name="M_PI" value="3.14159"/>
     <property name="HALF_PI" value="1.57079"/>
@@ -130,4 +131,6 @@
             <origin xyz="-0.14899868 0.17604938 -0.14899868" rpy="0 0 0"/>
         </xacro:pillar_plate>
+	<xacro:jaco2_custom base_parent="pillar_plate_link">
+	</xacro:jaco2_custom>
         <!-- Poli Sensors -->
         <xacro:hokuyo_ust30lx laser_prefix="${REAR_LASER_PREFIX}" parent="rmp_plate2_link">

Commit message: fixed location of parent links

File: poli2_description/robots/jaco2_custom.xacro (robot description, xacro)
@@ -101,5 +101,5 @@
     <property name="joint_end_effector_origin_xyz" value="0 0 -0.1600" />
     <property name="joint_end_effector_origin_rpy" value="${J_PI} 0 0" />
-    <xacro:macro name="jaco2_custom" params="base_origin_parent base_xyz base_origin_rpy prefix:=j2s7s300">
+    <xacro:macro name="jaco2_custom" params="base_parent base_origin_xyz base_origin_rpy prefix:=j2s7s300">
         <xacro:gazebo_config robot_namespace="${prefix}"/>
         <xacro:kinova_armlink link_name="${prefix}_link_base" link_mesh="${link_base_mesh}" mesh_no="${link_base_mesh_no}"/>

File: poli2_description/robots/poli.urdf.xacro (robot description, xacro)
@@ -131,5 +131,5 @@
             <origin xyz="-0.14899868 0.17604938 -0.14899868" rpy="0 0 0"/>
         </xacro:pillar_plate>
-	<xacro:jaco2_custom base_parent="pillar_plate_link">
+	<xacro:jaco2_custom base_parent="pillar_plate_link" base_origin_xyz="0 0 0" base_origin_rpy="-${HALF_PI} -${HALF_PI} 0">
 	</xacro:jaco2_custom>
         <!-- Poli Sensors -->

Commit message: Fix: Gripper and MoveIt! integration (#19)
* fixed wsg_50 param issue

* halfway adding jaco to robot

* fixed location of parent links

* copied standalone moveit configuration to the full robot

* modified collision geometries to be accurate according to mesh model. fixed wrist rotational issue wrt the model vs reality.

* fixed standalone description files for jaco2 custom

* renamed the standalone jaco moveit configuration

* regenerated urdf with changes in wsg_32_description. accurately shows finger movement

File: poli2_description/robots/jaco2_custom.xacro (robot description, xacro)
@@ -101,8 +101,8 @@
     <property name="joint_end_effector_origin_xyz" value="0 0 -0.1600" />
     <property name="joint_end_effector_origin_rpy" value="${J_PI} 0 0" />
-    <xacro:macro name="jaco2_custom" params="base_parent prefix:=j2s7s300">
+    <xacro:macro name="jaco2_custom" params="base_parent base_origin_xyz base_origin_rpy prefix:=j2s7s300">
         <xacro:gazebo_config robot_namespace="${prefix}"/>
         <xacro:kinova_armlink link_name="${prefix}_link_base" link_mesh="${link_base_mesh}" mesh_no="${link_base_mesh_no}"/>
-        <xacro:kinova_armjoint joint_name="${prefix}_joint_base" type="${joint_base_type}" parent="${base_parent}" child="${prefix}_link_base" joint_axis_xyz="${joint_base_axis_xyz}" joint_origin_xyz="${joint_base_origin_xyz}" joint_origin_rpy="${joint_base_origin_rpy}" joint_lower_limit="0" joint_upper_limit="0" fixed="true"/>
+        <xacro:kinova_armjoint joint_name="${prefix}_joint_base" type="${joint_base_type}" parent="${base_parent}" child="${prefix}_link_base" joint_axis_xyz="${joint_base_axis_xyz}" joint_origin_xyz="${base_origin_xyz}" joint_origin_rpy="${base_origin_rpy}" joint_lower_limit="0" joint_upper_limit="0" fixed="true"/>
         <xacro:kinova_armlink link_name="${prefix}_link_1" link_mesh="${link_1_mesh}" use_ring_mesh="true" mesh_no="${link_1_mesh_no}"/>
         <xacro:kinova_armjoint joint_name="${prefix}_joint_1" type="${joint_1_type}" parent="${prefix}_link_base" child="${prefix}_link_1" joint_axis_xyz="${joint_1_axis_xyz}" joint_origin_xyz="${joint_1_origin_xyz}" joint_origin_rpy="${joint_1_origin_rpy}" joint_lower_limit="${joint_1_lower_limit}" joint_upper_limit="${joint_1_upper_limit}"/>

File: poli2_description/robots/poli.urdf.xacro (robot description, xacro)
@@ -35,4 +35,5 @@
     <xacro:include filename="$(find poli2_description)/urdf/poli_components/pillar.urdf.xacro"/>
     <xacro:include filename="$(find poli2_description)/urdf/poli_components/pillar_plate.urdf.xacro"/>
+    <xacro:include filename="$(find poli2_description)/robots/jaco2_custom.xacro"/>
     <property name="M_PI" value="3.14159"/>
     <property name="HALF_PI" value="1.57079"/>
@@ -130,4 +131,6 @@
             <origin xyz="-0.14899868 0.17604938 -0.14899868" rpy="0 0 0"/>
         </xacro:pillar_plate>
+	<xacro:jaco2_custom base_parent="pillar_plate_link" base_origin_xyz="0 0 0" base_origin_rpy="-${HALF_PI} -${HALF_PI} 0">
+	</xacro:jaco2_custom>
         <!-- Poli Sensors -->
         <xacro:hokuyo_ust30lx laser_prefix="${REAR_LASER_PREFIX}" parent="rmp_plate2_link">

Commit message: added arm back to urdf and modified bringup scripts to publish arm state again

File: poli2_description/robots/jaco2_custom.xacro (robot description, xacro)
@@ -120,7 +120,7 @@
             <origin xyz="${joint_7_origin_xyz}" rpy="-${J_PI/2} 0 0"/>
         </xacro:weiss_mount>
-        <xacro:wsg_32_xacro name="wsg_50_gripper" parent="${prefix}_link_7">
+        <!--xacro:wsg_32_xacro name="wsg_50_gripper" parent="${prefix}_link_7">
             <origin xyz="0.0001 0 0.085" rpy="0 0 -${J_PI/2}"/>
-        </xacro:wsg_32_xacro>
+        </xacro:wsg_32_xacro-->
     </xacro:macro>
 </root>

File: poli2_description/robots/jaco2_custom_wrapper.urdf (robot description, URDF)
Before this commit: robot j2s7s300, 15 links, 14 joints
Links:
- removed link wsg_50_gripper_base_link
- removed link wsg_50_gripper_base_link_gripper_left
- removed link wsg_50_gripper_base_link_gripper_right
- removed link wsg_50_gripper_left_universal_finger_link
- removed link wsg_50_gripper_right_universal_finger_link
Joints:
- removed joint wsg_50_gripper_base_joint
- removed joint wsg_50_gripper_base_joint_gripper_left
- removed joint wsg_50_gripper_base_joint_gripper_right
- removed joint wsg_50_gripper_left_universal_finger_joint
- removed joint wsg_50_gripper_right_universal_finger_joint

File: poli2_description/robots/poli.urdf (robot description, URDF)
Before this commit: robot segway_robot, 45 links, 44 joints
Links:
- removed link wsg_50_gripper_base_link
- removed link wsg_50_gripper_base_link_gripper_left
- removed link wsg_50_gripper_base_link_gripper_right
- removed link wsg_50_gripper_left_universal_finger_link
- removed link wsg_50_gripper_right_universal_finger_link
- link neck_base_link: mass 0.557568366166049 -> 0.6796
- link pan_link: mass 0.661811908284221 -> 0.28209
- link tilt_link: mass 0.0557850572590686 -> 0.282648823094398
Joints:
- removed joint wsg_50_gripper_base_joint
- removed joint wsg_50_gripper_base_joint_gripper_left
- removed joint wsg_50_gripper_base_joint_gripper_right
- removed joint wsg_50_gripper_left_universal_finger_joint
- removed joint wsg_50_gripper_right_universal_finger_joint
- joint camera_rgb_joint: origin xyz=-0.08 -0.0035 0.05 rpy=0 0 3.14159 -> xyz=-0.22 0.0 -0.0624  rpy=1.57079 0 4.18879
- joint neck_base_joint: origin xyz=0.1785 0.385 0.205 rpy=0 0 1.57079 -> xyz=0.2658 0.36 0.1915 rpy=-1.57079 0 0
- joint pan_joint: axis 1 0 0 -> 0 0 1; limit lower=-1.54 upper=1.54 effort=30 velocity=1.0 -> lower=-1.54 upper=1.54 effort=10 velocity=10; origin xyz=0.0179 0 0 rpy=0 0 0 -> xyz=0.0014145 0 0.0466 rpy=0 0 0
- joint tilt_joint: axis 0 -1 0 -> 0 0 1; limit lower=-0.7 upper=0.8 effort=1.0 velocity=1.0 -> lower=-1.0471975512 upper=0.0 effort=10.0 velocity=1.0; origin xyz=0.1011 0 -0.00960000000000004 rpy=-1.5707963267949 0 -1.5707963267949 -> xyz=0 -0.05475 0.09675 rpy=1.5708 0 0

File: poli2_description/robots/poli.urdf.xacro (robot description, xacro)
@@ -137,8 +137,6 @@
             <origin xyz="0.2658 0.36 0.1915" rpy="-${HALF_PI} 0 0"/>
         </xacro:neck_mount>
-	<!--
 	<xacro:jaco2_custom base_parent="pillar_plate_link" base_origin_xyz="0 0.05 0.0575" base_origin_rpy="-${HALF_PI} -${HALF_PI} 0">
 	</xacro:jaco2_custom>
-        -->
         <!-- Poli Sensors -->
         <xacro:hokuyo_ust30lx laser_prefix="${REAR_LASER_PREFIX}" parent="rmp_plate2_link">

Commit message: added robotiq package and modified urdf and moveit for gripper

File: poli2_description/robots/jaco2_custom.xacro (robot description, xacro)
@@ -117,7 +117,20 @@
         <xacro:kinova_armlink link_name="${prefix}_link_6" link_mesh="${link_6_mesh}" use_ring_mesh="true" ring_mesh="ring_small" mesh_no="${link_6_mesh_no}"/>
         <xacro:kinova_armjoint joint_name="${prefix}_joint_6" type="${joint_6_type}" parent="${prefix}_link_5" child="${prefix}_link_6" joint_axis_xyz="${joint_6_axis_xyz}" joint_origin_xyz="${joint_6_origin_xyz}" joint_origin_rpy="${joint_6_origin_rpy}" joint_lower_limit="${joint_6_lower_limit}" joint_upper_limit="${joint_6_upper_limit}"/>
-        <xacro:weiss_mount link_name="${prefix}_link_7" joint_name="${prefix}_joint_7" parent="${prefix}_link_6">
+	<joint name="${prefix}ee_fixed_joint" type="fixed">
+            <parent link="${prefix}_link_6" />
+            <child link = "${prefix}ee_base" />
+            <origin xyz="0 0 -0.09380704" rpy="${M_PI} ${M_PI/2} 0" /> <!--0.09380704156-->
+        </joint>
+        <link name="${prefix}ee_base"/>
+        <!-- Add in an EEF link for the center of the gripper -->
+        <joint name="${prefix}ee_gripper" type="fixed">
+            <parent link="${prefix}ee_base" />
+            <child link ="${prefix}ee_link" />
+            <origin xyz="0.13 0 0" />
+        </joint>
+	<link name="${prefix}ee_link"/>
+        <!--xacro:weiss_mount link_name="${prefix}_link_7" joint_name="${prefix}_joint_7" parent="${prefix}_link_6">
             <origin xyz="${joint_7_origin_xyz}" rpy="-${J_PI/2} 0 0"/>
-        </xacro:weiss_mount>
+        </xacro:weiss_mount-->
         <!--xacro:wsg_32_xacro name="wsg_50_gripper" parent="${prefix}_link_7">
             <origin xyz="0.0001 0 0.085" rpy="0 0 -${J_PI/2}"/>

File: poli2_description/robots/poli.urdf (robot description, URDF)
Before this commit: robot segway_robot, 40 links, 39 joints
Links:
- added link gripper_base_link, mass 0.636951; collision mesh filename=package://robotiq_85_description/meshes/collision/robotiq_8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; visual mesh filename=package://robotiq_85_description/meshes/visual/robotiq_85_b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
- added link gripper_finger1_finger_link, mass 0.027309; collision mesh filename=package://robotiq_85_description/meshes/collision/robotiq_8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; visual mesh filename=package://robotiq_85_description/meshes/visual/robotiq_85_f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
- added link gripper_finger1_finger_tip_link, mass 0.019555; collision mesh filename=package://robotiq_85_description/meshes/collision/robotiq_8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; visual mesh filename=package://robotiq_85_description/meshes/visual/robotiq_85_f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
- added link gripper_finger1_inner_knuckle_link, mass 0.029951; collision mesh filename=package://robotiq_85_description/meshes/collision/robotiq_8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; visual mesh filename=package://robotiq_85_description/meshes/visual/robotiq_85_i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
- added link gripper_finger1_knuckle_link, mass 0.018491; collision mesh filename=package://robotiq_85_description/meshes/collision/robotiq_8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; visual mesh filename=package://robotiq_85_description/meshes/visual/robotiq_85_k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
- added link gripper_finger2_finger_link, mass 0.027309; collision mesh filename=package://robotiq_85_description/meshes/collision/robotiq_8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; visual mesh filename=package://robotiq_85_description/meshes/visual/robotiq_85_f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
- added link gripper_finger2_finger_tip_link, mass 0.019555; collision mesh filename=package://robotiq_85_description/meshes/collision/robotiq_8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; visual mesh filename=package://robotiq_85_description/meshes/visual/robotiq_85_f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
- added link gripper_finger2_inner_knuckle_link, mass 0.029951; collision mesh filename=package://robotiq_85_description/meshes/collision/robotiq_8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; visual mesh filename=package://robotiq_85_description/meshes/visual/robotiq_85_i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
- added link gripper_finger2_knuckle_link, mass 0.018491; collision mesh filename=package://robotiq_85_description/meshes/collision/robotiq_8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; visual mesh filename=package://robotiq_85_description/meshes/visual/robotiq_85_k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
- added link j2s7s300_ee_base
- added link j2s7s300_ee_link
- link j2s7s300_link_7: geometry collision mesh filename=package://kinova_description/meshes/wrist_3.stl; visual mesh filename=package://kinova_description/meshes/wrist_3.dae
Joints:
- added joint gripper_base_joint: type fixed, parent j2s7s300_ee_base, child gripper_base_link, origin xyz=0 0 0 rpy=0 0 0
- added joint gripper_finger1_finger_joint: type fixed, parent gripper_finger1_knuckle_link, child gripper_finger1_finger_link, origin xyz=-0.00408552455 -0.03148604435 0.0 rpy=0 0 0
- added joint gripper_finger1_finger_tip_joint: type continuous, parent gripper_finger1_inner_knuckle_link, child gripper_finger1_finger_tip_link, origin xyz=0.04303959807 -0.03759940821 0.0 rpy=0.0 0.0 0.0, axis 0 0 1, limit lower=-3.14 upper=3.14 effort=0.1 velocity=100.0, mimic joint=gripper_finger1_joint multiplier=-1
- added joint gripper_finger1_inner_knuckle_joint: type continuous, parent gripper_base_link, child gripper_finger1_inner_knuckle_link, origin xyz=0.06142 0.0127 0 rpy=3.14159265359 0.0 0.0, axis 0 0 1, limit lower=-3.14 upper=3.14 effort=0.1 velocity=100.0, mimic joint=gripper_finger1_joint offset=0
- added joint gripper_finger1_joint: type revolute, parent gripper_base_link, child gripper_finger1_knuckle_link, origin xyz=0.05490451627 0.03060114443 0.0 rpy=3.14159265359 0.0 0.0, axis 0 0 1, limit lower=0.0 upper=0.804 effort=1000 velocity=2.0
- added joint gripper_finger2_finger_joint: type fixed, parent gripper_finger2_knuckle_link, child gripper_finger2_finger_link, origin xyz=-0.00408552455 -0.03148604435 0.0 rpy=0 0 0
- added joint gripper_finger2_finger_tip_joint: type continuous, parent gripper_finger2_inner_knuckle_link, child gripper_finger2_finger_tip_link, origin xyz=0.04303959807 -0.03759940821  0.0 rpy=0.0 0.0 0.0, axis 0 0 1, limit lower=-3.14 upper=3.14 effort=0.1 velocity=100.0, mimic joint=gripper_finger1_joint multiplier=-1
- added joint gripper_finger2_inner_knuckle_joint: type continuous, parent gripper_base_link, child gripper_finger2_inner_knuckle_link, origin xyz=0.06142 -0.0127 0 rpy=0 0 0, axis 0 0 1, limit lower=-3.14 upper=3.14 effort=0.1 velocity=100.0, mimic joint=gripper_finger1_joint offset=0
- added joint gripper_finger2_joint: type revolute, parent gripper_base_link, child gripper_finger2_knuckle_link, origin xyz=0.05490451627 -0.03060114443 0.0 rpy=0.0 0.0 0.0, axis 0 0 1, limit lower=-3.14 upper=3.14 effort=1000 velocity=100.0, mimic joint=gripper_finger1_joint
- added joint j2s7s300_ee_fixed_joint: type fixed, parent j2s7s300_link_7, child j2s7s300_ee_base, origin xyz=0 0 -0.09380704 rpy=0 1.57079632679 0
- added joint j2s7s300_ee_gripper: type fixed, parent j2s7s300_ee_base, child j2s7s300_ee_link, origin xyz=0.13 0 0
- joint j2s7s300_joint_7: axis 0 0 -1 -> 0 0 1; limit effort=50 velocity=50 -> effort=600.8 velocity=0.785; origin xyz=0 0.10375 0 rpy=-1.57079632679 0 0 -> xyz=0 0.06075 0 rpy=1.57079632679 0 0

File: poli2_description/robots/poli.urdf.xacro (robot description, xacro)
@@ -39,4 +39,5 @@
     <xacro:include filename="$(find poli2_description)/urdf/poli_components/neck_mount.urdf.xacro"/>
     <xacro:include filename="$(find poli2_description)/robots/jaco2_custom.xacro"/>
+    <xacro:include filename="$(find kinova_description)/urdf/j2s7s300.xacro" />
     <property name="M_PI" value="3.14159"/>
     <property name="HALF_PI" value="1.57079"/>
@@ -137,6 +138,7 @@
             <origin xyz="0.2658 0.36 0.1915" rpy="-${HALF_PI} 0 0"/>
         </xacro:neck_mount>
-	<xacro:jaco2_custom base_parent="pillar_plate_link" base_origin_xyz="0 0.05 0.0575" base_origin_rpy="-${HALF_PI} -${HALF_PI} 0">
-	</xacro:jaco2_custom>
+	<!-- Poli Jaco Arm -->
+	<xacro:j2s7s300 base_parent="pillar_plate_link" trans="0 0.05 0.0575" rot="-${HALF_PI} -${HALF_PI} 0">
+	</xacro:j2s7s300>
         <!-- Poli Sensors -->
         <xacro:hokuyo_ust30lx laser_prefix="${REAR_LASER_PREFIX}" parent="rmp_plate2_link">
