Commit message: added simulation files. added working movebase

File: poli2_description/robots/poli.urdf.xacro (robot description, xacro)
@@ -49,4 +49,15 @@
           <plugin name="gazebo_ros_control" filename="libgazebo_ros_control.so">
               <robotNamespace>/</robotNamespace>
+          </plugin>
+            <plugin name="object_controller" filename="libgazebo_ros_force_based_move.so">
+                <commandTopic>/cmd_vel</commandTopic>
+                <odometryTopic>/odom</odometryTopic>
+                <odometryFrame>odom</odometryFrame>
+                <odometryRate>30.0</odometryRate>
+                <robotBaseFrame>base_link</robotBaseFrame>
+                <publishOdometryTf>1</publishOdometryTf>
+                <yaw_velocity_p_gain>100.0</yaw_velocity_p_gain>
+                <x_velocity_p_gain>10000.0</x_velocity_p_gain>
+                <y_velocity_p_gain>10000.0</y_velocity_p_gain>
           </plugin>
         </gazebo>

File: poli2_description/urdf/poli_components/pillar.urdf.xacro (robot description, xacro)
@@ -39,5 +39,5 @@
             </collision>
         </link>
-        <joint name="pillar_telescope_joint" type="prismatic">
+        <joint name="pillar_telescope_joint" type="fixed">
             <origin xyz="0.2175586 0.1 0.02" rpy="0 -1.570796 0"/>
             <parent link="${parent}" />

Commit message: fixed orientation issue with base and lasers

File: poli2_description/robots/poli.urdf.xacro (robot description, xacro)
@@ -66,5 +66,5 @@
         <!--Chassis -->
         <xacro:powerbase_110 chassis_prefix="base" parent="base_link">
-            <origin xyz="0 0 ${-wheel_vertical_offset + wheel_radius}" rpy="0 0 0" />
+            <origin xyz="0 0 ${-wheel_vertical_offset + wheel_radius}" rpy="0 0 ${M_PI}" />
         </xacro:powerbase_110>
         <link name="inertial_collision_link">
@@ -131,8 +131,8 @@
         </xacro:pillar_plate>
         <!-- Poli Sensors -->
-        <xacro:hokuyo_ust30lx laser_prefix="${FRONT_LASER_PREFIX}" parent="rmp_plate2_link">
+        <xacro:hokuyo_ust30lx laser_prefix="${REAR_LASER_PREFIX}" parent="rmp_plate2_link">
             <origin xyz="0.242 0.075 0.33" rpy="-${HALF_PI} -${HALF_PI} 0" />
         </xacro:hokuyo_ust30lx>
-        <xacro:hokuyo_ust10lx laser_prefix="${REAR_LASER_PREFIX}" parent="rmp_plate3_link">
+        <xacro:hokuyo_ust10lx laser_prefix="${FRONT_LASER_PREFIX}" parent="rmp_plate3_link">
             <origin xyz="0.242 -0.015 0.33" rpy="${HALF_PI} -${HALF_PI} 0" />
         </xacro:hokuyo_ust10lx>

Commit message: fixed teleop / autonom navigation odometry issue

File: poli2_description/robots/poli.urdf.xacro (robot description, xacro)
@@ -66,5 +66,5 @@
         <!--Chassis -->
         <xacro:powerbase_110 chassis_prefix="base" parent="base_link">
-            <origin xyz="0 0 ${-wheel_vertical_offset + wheel_radius}" rpy="0 0 ${M_PI}" />
+            <origin xyz="0 0 ${-wheel_vertical_offset + wheel_radius}" rpy="0 0 0" />
         </xacro:powerbase_110>
         <link name="inertial_collision_link">

Commit message: added neck mount xacro files. Also added material for other stl files to increase contrast

File: poli2_description/robots/poli.urdf.xacro (robot description, xacro)
@@ -35,4 +35,5 @@
     <xacro:include filename="$(find poli2_description)/urdf/poli_components/pillar.urdf.xacro"/>
     <xacro:include filename="$(find poli2_description)/urdf/poli_components/pillar_plate.urdf.xacro"/>
+    <xacro:include filename="$(find poli2_description)/urdf/poli_components/neck_mount.urdf.xacro"/>
     <property name="M_PI" value="3.14159"/>
     <property name="HALF_PI" value="1.57079"/>
@@ -121,4 +122,7 @@
             <origin xyz="-0.14899868 0.17604938 -0.14899868" rpy="0 0 0"/>
         </xacro:pillar_plate>
+        <xacro:neck_mount parent="pillar_plate_link">
+            <origin xyz="0.22 0.385 0.19" rpy="0 0 ${HALF_PI}"/>
+        </xacro:neck_mount>
         <!-- Poli Sensors -->
         <xacro:hokuyo_ust30lx laser_prefix="${FRONT_LASER_PREFIX}" parent="rmp_plate2_link">

File: poli2_description/urdf/poli_components/base_plate.urdf.xacro (robot description, xacro)
@@ -32,4 +32,7 @@
                     <mesh filename="package://poli2_description/meshes/components/base_plate.STL" />
                 </geometry>
+                <material name="">
+                    <color rgba="0.5 0.5 0.5 1" />
+                </material>
             </visual>
             <collision>

File: poli2_description/urdf/poli_components/pillar.urdf.xacro (robot description, xacro)
@@ -32,4 +32,7 @@
                     <mesh filename="package://poli2_description/meshes/components/pillar_exterior.STL" />
                 </geometry>
+                <material name="">
+                    <color rgba="0.75 0.75 0.75 1" />
+                </material>
             </visual>
             <collision>
@@ -51,4 +54,7 @@
                     <mesh filename="package://poli2_description/meshes/components/pillar_telescope.STL" />
                 </geometry>
+                <material name="">
+                    <color rgba="0.3 0.3 0.3 1" />
+                </material>
             </visual>
             <collision>

File: poli2_description/urdf/poli_components/pillar_plate.urdf.xacro (robot description, xacro)
@@ -32,4 +32,7 @@
                     <mesh filename="package://poli2_description/meshes/components/pillar_plate.STL" />
                 </geometry>
+                <material name="">
+                    <color rgba="0.5 0.5 0.5 1" />
+                </material>
             </visual>
             <collision>

File: poli2_description/urdf/poli_components/rmp_plate2.urdf.xacro (robot description, xacro)
@@ -32,4 +32,7 @@
                     <mesh filename="package://poli2_description/meshes/components/rmp_plate2.STL" />
                 </geometry>
+            <material name="">
+                <color rgba="0.5 0.5 0.5 1" />
+            </material>
             </visual>
             <collision>

File: poli2_description/urdf/poli_components/rmp_plate3.urdf.xacro (robot description, xacro)
@@ -32,4 +32,7 @@
                     <mesh filename="package://poli2_description/meshes/components/rmp_plate3.STL" />
                 </geometry>
+                <material name="">
+                    <color rgba="0.5 0.5 0.5 1" />
+                </material>
             </visual>
             <collision>

Commit message: ros controller additions to make epos_hardware compatible. changes to make urdf work on robot

File: poli2_description/robots/poli.urdf.xacro (robot description, xacro)
@@ -105,6 +105,4 @@
             <origin xyz="0.32784550 0 0.03326933" rpy="0 0 0" />
         </xacro:caster_assembly_110>
-        <!-- Setup any accessories defined in the environment -->
-        <xacro:segway_accessories />
         <xacro:base_plate parent="base_chassis_link">
             <origin xyz="0.0762 0.16355 0.076" rpy="${HALF_PI} 0 -${HALF_PI}"/>

File: poli2_description/urdf/poli_components/neck_mount.urdf.xacro (robot description, xacro)
@@ -173,4 +173,11 @@
       xyz="0 1 0" />
   </joint>
+  <transmission name="tilt_joint_trans">
+    <type>transmission_interface/SimpleTransmission</type>
+    <joint name="tilt_joint">
+      <hardwareInterface>hardware_interface/PositionJointInterface</hardwareInterface>
+    </joint>
+    <actuator name="tilt_joint_actuator"></actuator>
+  </transmission>
     </xacro:macro>
 </robot>

Commit message: Feature/pan tilt integration (#21)
* added neck mount xacro files. Also added material for other stl files to increase contrast

* ros controller additions to make epos_hardware compatible. changes to make urdf work on robot

* added a few parameters

* updated parameters from windows software

* final parameter fixes. works!

* added position control capabilities from dynamixel tutorials

* merge residual

* changes to make state readable by tf

* fixed gear ratio for tilt. consolidated files

* residuals

* added proper handling of joint states

* made pan code consistent with tilt controller in namespace and command interface

* corrected joint limits for assumed starting position for tilt

* fixed joint limits for pan; joint state mapping; regenerated moveit config with pan_tilt

File: poli2_description/robots/poli.urdf.xacro (robot description, xacro)
@@ -35,4 +35,5 @@
     <xacro:include filename="$(find poli2_description)/urdf/poli_components/pillar.urdf.xacro"/>
     <xacro:include filename="$(find poli2_description)/urdf/poli_components/pillar_plate.urdf.xacro"/>
+    <xacro:include filename="$(find poli2_description)/urdf/poli_components/neck_mount.urdf.xacro"/>
     <xacro:include filename="$(find poli2_description)/robots/jaco2_custom.xacro"/>
     <property name="M_PI" value="3.14159"/>
@@ -131,4 +132,7 @@
             <origin xyz="-0.14899868 0.17604938 -0.14899868" rpy="0 0 0"/>
         </xacro:pillar_plate>
+        <xacro:neck_mount parent="pillar_plate_link">
+            <origin xyz="0.22 0.385 0.19" rpy="0 0 ${HALF_PI}"/>
+        </xacro:neck_mount>
 	<xacro:jaco2_custom base_parent="pillar_plate_link" base_origin_xyz="0 0 0" base_origin_rpy="-${HALF_PI} -${HALF_PI} 0">
 	</xacro:jaco2_custom>

File: poli2_description/urdf/poli_components/base_plate.urdf.xacro (robot description, xacro)
@@ -32,4 +32,7 @@
                     <mesh filename="package://poli2_description/meshes/components/base_plate.STL" />
                 </geometry>
+                <material name="">
+                    <color rgba="0.5 0.5 0.5 1" />
+                </material>
             </visual>
             <collision>

File: poli2_description/urdf/poli_components/pillar.urdf.xacro (robot description, xacro)
@@ -32,4 +32,7 @@
                     <mesh filename="package://poli2_description/meshes/components/pillar_exterior.STL" />
                 </geometry>
+                <material name="">
+                    <color rgba="0.75 0.75 0.75 1" />
+                </material>
             </visual>
             <collision>
@@ -51,4 +54,7 @@
                     <mesh filename="package://poli2_description/meshes/components/pillar_telescope.STL" />
                 </geometry>
+                <material name="">
+                    <color rgba="0.3 0.3 0.3 1" />
+                </material>
             </visual>
             <collision>

File: poli2_description/urdf/poli_components/pillar_plate.urdf.xacro (robot description, xacro)
@@ -32,4 +32,7 @@
                     <mesh filename="package://poli2_description/meshes/components/pillar_plate.STL" />
                 </geometry>
+                <material name="">
+                    <color rgba="0.5 0.5 0.5 1" />
+                </material>
             </visual>
             <collision>

File: poli2_description/urdf/poli_components/rmp_plate2.urdf.xacro (robot description, xacro)
@@ -32,4 +32,7 @@
                     <mesh filename="package://poli2_description/meshes/components/rmp_plate2.STL" />
                 </geometry>
+            <material name="">
+                <color rgba="0.5 0.5 0.5 1" />
+            </material>
             </visual>
             <collision>

File: poli2_description/urdf/poli_components/rmp_plate3.urdf.xacro (robot description, xacro)
@@ -32,4 +32,7 @@
                     <mesh filename="package://poli2_description/meshes/components/rmp_plate3.STL" />
                 </geometry>
+                <material name="">
+                    <color rgba="0.5 0.5 0.5 1" />
+                </material>
             </visual>
             <collision>

Commit message: added sonar to urdf model. sonar arduino driver

File: poli2_description/robots/poli.urdf.xacro (robot description, xacro)
@@ -31,4 +31,5 @@
     <xacro:include filename="$(find poli2_description)/urdf/sensors/hokuyo_ust30lx.urdf.xacro"/>
     <xacro:include filename="$(find poli2_description)/urdf/sensors/astra.urdf.xacro"/>
+    <xacro:include filename="$(find poli2_description)/urdf/sensors/sonar.urdf.xacro"/>
     <xacro:include filename="$(find poli2_description)/urdf/poli_components/base_plate.urdf.xacro"/>
     <xacro:include filename="$(find poli2_description)/urdf/poli_components/rmp_plate2.urdf.xacro"/>
@@ -148,4 +149,7 @@
 	    <origin xyz="-0.08 -0.0035 0.05" rpy="0 0 ${M_PI}"/>
         </xacro:sensor_astra>
+        <xacro:sensor_sonar parent="pillar_plate_link">
+            <origin xyz="0.007 0.022 0.203" rpy="${HALF_PI} 0 ${HALF_PI}"/>
+        </xacro:sensor_sonar>
     </xacro:macro>
 </robot>

Commit message: Sonar + range navigation (#25)
* poli1 upstart additions

* poli2 upstart additions

* changed model axis of rotation to match actuator

* added sonar to urdf model. sonar arduino driver

* added sonar into navigation

* fixed tf and baud rate issues

* added planner?

* tf and navigation tweaks

* added max range limit for obstacle range clearing

File: poli2_description/robots/poli.urdf.xacro (robot description, xacro)
@@ -31,4 +31,5 @@
     <xacro:include filename="$(find poli2_description)/urdf/sensors/hokuyo_ust30lx.urdf.xacro"/>
     <xacro:include filename="$(find poli2_description)/urdf/sensors/astra.urdf.xacro"/>
+    <xacro:include filename="$(find poli2_description)/urdf/sensors/sonar.urdf.xacro"/>
     <xacro:include filename="$(find poli2_description)/urdf/poli_components/base_plate.urdf.xacro"/>
     <xacro:include filename="$(find poli2_description)/urdf/poli_components/rmp_plate2.urdf.xacro"/>
@@ -148,4 +149,7 @@
 	    <origin xyz="-0.08 -0.0035 0.05" rpy="0 0 ${M_PI}"/>
         </xacro:sensor_astra>
+        <xacro:sensor_sonar parent="pillar_plate_link">
+            <origin xyz="0.007 0.022 0.203" rpy="${HALF_PI} 0 ${HALF_PI*2}"/>
+        </xacro:sensor_sonar>
     </xacro:macro>
 </robot>

Commit message: updates the neck assembly to final beta version. changes movement angle to correct 60 degrees

File: poli2_description/robots/poli.urdf.xacro (robot description, xacro)
@@ -135,5 +135,5 @@
         </xacro:pillar_plate>
         <xacro:neck_mount parent="pillar_plate_link">
-            <origin xyz="0.1785 0.385 0.205" rpy="0 0 ${HALF_PI}"/>
+            <origin xyz="0.1785 0.385 0.205" rpy="-${HALF_PI} 0 0"/>
         </xacro:neck_mount>
 	<xacro:jaco2_custom base_parent="pillar_plate_link" base_origin_xyz="0 0.05 0.0575" base_origin_rpy="-${HALF_PI} -${HALF_PI} 0">
@@ -147,5 +147,5 @@
         </xacro:hokuyo_ust10lx>
         <xacro:sensor_astra parent="tilt_link">
-	    <origin xyz="-0.08 -0.0035 0.05" rpy="0 0 ${M_PI}"/>
+	    <origin xyz="-0.22 0.0 -0.0624 " rpy="${HALF_PI} 0 ${M_PI+1.0472}"/>
         </xacro:sensor_astra>
         <xacro:sensor_sonar parent="pillar_plate_link">

File: poli2_description/urdf/poli_components/neck_mount.urdf.xacro (robot description, xacro)
@@ -31,15 +31,15 @@
     <inertial>
       <origin
-        xyz="0.0148515762658108 -0.00184105590397508 -0.000758781648758649"
+        xyz="0.0023997 -3.3244E-06 0.033447"
         rpy="0 0 0" />
       <mass
-        value="0.557568366166049" />
+        value="0.6796" />
       <inertia
-        ixx="0.000397280277578404"
-        ixy="-1.20167051949868E-05"
-        ixz="-1.63630013884179E-05"
-        iyy="0.000682280271694407"
-        iyz="7.78900389369296E-07"
-        izz="0.000735555743930346" />
+        ixx="0.0014012"
+        ixy="9.4856E-09"
+        ixz="-3.5218E-06"
+        iyy="0.0010212"
+        iyz="-7.8472E-10"
+        izz="0.0010421" />
     </inertial>
     <visual>
@@ -54,5 +54,5 @@
         name="">
         <color
-          rgba="0.776470588235294 0.756862745098039 0.737254901960784 1" />
+          rgba="0.89804 0.91765 0.92941 1" />
       </material>
     </visual>
@@ -66,20 +66,20 @@
       </geometry>
     </collision>
-  </link>
-  <link
+   </link>
+   <link
     name="pan_link">
     <inertial>
       <origin
-        xyz="0.0864835918741103 0.000240681934725141 -0.00112944538944813"
+        xyz="-0.00034561 -0.0064887 0.077201"
         rpy="0 0 0" />
       <mass
-        value="0.661811908284221" />
+        value="0.28209" />
       <inertia
-        ixx="0.000586217271198065"
-        ixy="-2.32821859823434E-06"
-        ixz="1.20338819263342E-05"
-        iyy="0.000978190133235562"
-        iyz="3.81415623052038E-06"
-        izz="0.000579159076299907" />
+        ixx="0.00045437"
+        ixy="-3.8199E-06"
+        ixz="2.945E-06"
+        iyy="0.00019445"
+        iyz="3.612E-05"
+        izz="0.00032985" />
     </inertial>
     <visual>
@@ -94,5 +94,5 @@
         name="">
         <color
-          rgba="0.898039215686275 0.917647058823529 0.929411764705882 1" />
+          rgba="0.89804 0.91765 0.92941 1" />
       </material>
     </visual>
@@ -110,7 +110,7 @@
     name="pan_joint"
     type="revolute">
-    <limit lower="-1.54" upper="1.54" velocity="1.0" effort="30"/>
+    <limit lower="-1.54" upper="1.54" velocity="10" effort="10"/>
     <origin
-      xyz="0.0179 0 0"
+      xyz="0.0014145 0 0.0466"
       rpy="0 0 0" />
     <parent
@@ -119,5 +119,5 @@
       link="pan_link" />
     <axis
-      xyz="1 0 0" />
+      xyz="0 0 -1" />
   </joint>
   <link
@@ -125,15 +125,15 @@
     <inertial>
       <origin
-        xyz="-0.0466008886423734 -0.00905441755654412 -0.000748921866620636"
+        xyz="-0.0449449011423384 0.0505307759460616 -0.0582731595130051"
         rpy="0 0 0" />
       <mass
-        value="0.0557850572590686" />
+        value="0.282648823094398" />
       <inertia
-        ixx="7.04408522869088E-05"
-        ixy="-1.418314255844E-06"
-        ixz="-5.5662147711043E-07"
-        iyy="4.66839851062126E-05"
-        iyz="-2.27936975213634E-08"
-        izz="0.000115169958191947" />
+        ixx="0.000800089809159035"
+        ixy="0.000149569968914255"
+        ixz="4.25601989889811E-05"
+        iyy="0.00166070452096634"
+        iyz="-5.10288056116621E-05"
+        izz="0.00151354802293456" />
     </inertial>
     <visual>
@@ -148,5 +148,5 @@
         name="">
         <color
-          rgba="0.5 0.5 0.5 1" />
+          rgba="0.898039215686275 0.917647058823529 0.929411764705882 1" />
       </material>
     </visual>
@@ -164,8 +164,8 @@
     name="tilt_joint"
     type="revolute">
-    <limit lower="-0.7" upper="0.8" velocity="1.0" effort="1.0"/>
+    <limit lower="0.0" upper="1.0471975512" velocity="1.0" effort="1.0"/>
     <origin
-      xyz="0.1011 0 -0.00960000000000004"
-      rpy="-1.5707963267949 0 -1.5707963267949" />
+      xyz="0 -0.05475 0.09675"
+      rpy="1.5708 0 0" />
     <parent
       link="pan_link" />
@@ -173,5 +173,5 @@
       link="tilt_link" />
     <axis
-      xyz="0 -1 0" />
+      xyz="0 0 1" />
   </joint>
   <transmission name="tilt_joint_trans">
@@ -184,4 +184,4 @@
     </actuator>
   </transmission>
-    </xacro:macro>
+  </xacro:macro>
 </robot>

Commit message: neck mount movement

File: poli2_description/robots/poli.urdf.xacro (robot description, xacro)
@@ -135,5 +135,5 @@
         </xacro:pillar_plate>
         <xacro:neck_mount parent="pillar_plate_link">
-            <origin xyz="0.1785 0.385 0.205" rpy="-${HALF_PI} 0 0"/>
+            <origin xyz="0.2658 0.36 0.1915" rpy="-${HALF_PI} 0 0"/>
         </xacro:neck_mount>
 	<xacro:jaco2_custom base_parent="pillar_plate_link" base_origin_xyz="0 0.05 0.0575" base_origin_rpy="-${HALF_PI} -${HALF_PI} 0">

File: poli2_description/urdf/poli_components/neck_mount.urdf.xacro (robot description, xacro)
@@ -173,5 +173,5 @@
       link="tilt_link" />
     <axis
-      xyz="0 0 1" />
+      xyz="0 0 -1" />
   </joint>
   <transmission name="tilt_joint_trans">

Commit message: corrections to axes of rotations and limits to match actual motor system

File: poli2_description/robots/poli.urdf.xacro (robot description, xacro)
@@ -137,6 +137,8 @@
             <origin xyz="0.2658 0.36 0.1915" rpy="-${HALF_PI} 0 0"/>
         </xacro:neck_mount>
+	<!--
 	<xacro:jaco2_custom base_parent="pillar_plate_link" base_origin_xyz="0 0.05 0.0575" base_origin_rpy="-${HALF_PI} -${HALF_PI} 0">
 	</xacro:jaco2_custom>
+        -->
         <!-- Poli Sensors -->
         <xacro:hokuyo_ust30lx laser_prefix="${REAR_LASER_PREFIX}" parent="rmp_plate2_link">

File: poli2_description/urdf/poli_components/neck_mount.urdf.xacro (robot description, xacro)
@@ -119,5 +119,5 @@
       link="pan_link" />
     <axis
-      xyz="0 0 -1" />
+      xyz="0 0 1" />
   </joint>
   <link
@@ -164,5 +164,5 @@
     name="tilt_joint"
     type="revolute">
-    <limit lower="0.0" upper="1.0471975512" velocity="1.0" effort="1.0"/>
+    <limit upper="0.0" lower="-1.0471975512" velocity="1.0" effort="10.0"/>
     <origin
       xyz="0 -0.05475 0.09675"
@@ -173,5 +173,5 @@
       link="tilt_link" />
     <axis
-      xyz="0 0 -1" />
+      xyz="0 0 1" />
   </joint>
   <transmission name="tilt_joint_trans">
