Commit message: LED controller, limit switch (#36)
* updates the neck assembly to final beta version. changes movement angle to correct 60 degrees

* neck mount movement

* corrections to axes of rotations and limits to match actual motor system

* removed arm and wsg gripper from higher level launch files

* modified port names due to new devices. added led controller launch file.

* corrected baud rate

* adds a high level driver that verifies correct starting position of tilt motor

* added missing led ino file and required msgs

* fixes for switch to arduino Mega. stable, but a few methods do not work

* fixes broken methods. allows ear led pulsing and a blinking method without blocking calls

* adds a startup script as per #32

* adds movement script as part of launch sequence

* added missing pulsing trigger

* small changes to improve readability on launch

File: poli2_description/robots/poli.urdf.xacro (robot description, xacro)
@@ -135,8 +135,10 @@
         </xacro:pillar_plate>
         <xacro:neck_mount parent="pillar_plate_link">
-            <origin xyz="0.1785 0.385 0.205" rpy="0 0 ${HALF_PI}"/>
+            <origin xyz="0.2658 0.36 0.1915" rpy="-${HALF_PI} 0 0"/>
         </xacro:neck_mount>
+	<!--
 	<xacro:jaco2_custom base_parent="pillar_plate_link" base_origin_xyz="0 0.05 0.0575" base_origin_rpy="-${HALF_PI} -${HALF_PI} 0">
 	</xacro:jaco2_custom>
+        -->
         <!-- Poli Sensors -->
         <xacro:hokuyo_ust30lx laser_prefix="${REAR_LASER_PREFIX}" parent="rmp_plate2_link">
@@ -147,5 +149,5 @@
         </xacro:hokuyo_ust10lx>
         <xacro:sensor_astra parent="tilt_link">
-	    <origin xyz="-0.08 -0.0035 0.05" rpy="0 0 ${M_PI}"/>
+	    <origin xyz="-0.22 0.0 -0.0624 " rpy="${HALF_PI} 0 ${M_PI+1.0472}"/>
         </xacro:sensor_astra>
         <xacro:sensor_sonar parent="pillar_plate_link">

File: poli2_description/urdf/poli_components/neck_mount.urdf.xacro (robot description, xacro)
@@ -31,15 +31,15 @@
     <inertial>
       <origin
-        xyz="0.0148515762658108 -0.00184105590397508 -0.000758781648758649"
+        xyz="0.0023997 -3.3244E-06 0.033447"
         rpy="0 0 0" />
       <mass
-        value="0.557568366166049" />
+        value="0.6796" />
       <inertia
-        ixx="0.000397280277578404"
-        ixy="-1.20167051949868E-05"
-        ixz="-1.63630013884179E-05"
-        iyy="0.000682280271694407"
-        iyz="7.78900389369296E-07"
-        izz="0.000735555743930346" />
+        ixx="0.0014012"
+        ixy="9.4856E-09"
+        ixz="-3.5218E-06"
+        iyy="0.0010212"
+        iyz="-7.8472E-10"
+        izz="0.0010421" />
     </inertial>
     <visual>
@@ -54,5 +54,5 @@
         name="">
         <color
-          rgba="0.776470588235294 0.756862745098039 0.737254901960784 1" />
+          rgba="0.89804 0.91765 0.92941 1" />
       </material>
     </visual>
@@ -66,20 +66,20 @@
       </geometry>
     </collision>
-  </link>
-  <link
+   </link>
+   <link
     name="pan_link">
     <inertial>
       <origin
-        xyz="0.0864835918741103 0.000240681934725141 -0.00112944538944813"
+        xyz="-0.00034561 -0.0064887 0.077201"
         rpy="0 0 0" />
       <mass
-        value="0.661811908284221" />
+        value="0.28209" />
       <inertia
-        ixx="0.000586217271198065"
-        ixy="-2.32821859823434E-06"
-        ixz="1.20338819263342E-05"
-        iyy="0.000978190133235562"
-        iyz="3.81415623052038E-06"
-        izz="0.000579159076299907" />
+        ixx="0.00045437"
+        ixy="-3.8199E-06"
+        ixz="2.945E-06"
+        iyy="0.00019445"
+        iyz="3.612E-05"
+        izz="0.00032985" />
     </inertial>
     <visual>
@@ -94,5 +94,5 @@
         name="">
         <color
-          rgba="0.898039215686275 0.917647058823529 0.929411764705882 1" />
+          rgba="0.89804 0.91765 0.92941 1" />
       </material>
     </visual>
@@ -110,7 +110,7 @@
     name="pan_joint"
     type="revolute">
-    <limit lower="-1.54" upper="1.54" velocity="1.0" effort="30"/>
+    <limit lower="-1.54" upper="1.54" velocity="10" effort="10"/>
     <origin
-      xyz="0.0179 0 0"
+      xyz="0.0014145 0 0.0466"
       rpy="0 0 0" />
     <parent
@@ -119,5 +119,5 @@
       link="pan_link" />
     <axis
-      xyz="1 0 0" />
+      xyz="0 0 1" />
   </joint>
   <link
@@ -125,15 +125,15 @@
     <inertial>
       <origin
-        xyz="-0.0466008886423734 -0.00905441755654412 -0.000748921866620636"
+        xyz="-0.0449449011423384 0.0505307759460616 -0.0582731595130051"
         rpy="0 0 0" />
       <mass
-        value="0.0557850572590686" />
+        value="0.282648823094398" />
       <inertia
-        ixx="7.04408522869088E-05"
-        ixy="-1.418314255844E-06"
-        ixz="-5.5662147711043E-07"
-        iyy="4.66839851062126E-05"
-        iyz="-2.27936975213634E-08"
-        izz="0.000115169958191947" />
+        ixx="0.000800089809159035"
+        ixy="0.000149569968914255"
+        ixz="4.25601989889811E-05"
+        iyy="0.00166070452096634"
+        iyz="-5.10288056116621E-05"
+        izz="0.00151354802293456" />
     </inertial>
     <visual>
@@ -148,5 +148,5 @@
         name="">
         <color
-          rgba="0.5 0.5 0.5 1" />
+          rgba="0.898039215686275 0.917647058823529 0.929411764705882 1" />
       </material>
     </visual>
@@ -164,8 +164,8 @@
     name="tilt_joint"
     type="revolute">
-    <limit lower="-0.7" upper="0.8" velocity="1.0" effort="1.0"/>
+    <limit upper="0.0" lower="-1.0471975512" velocity="1.0" effort="10.0"/>
     <origin
-      xyz="0.1011 0 -0.00960000000000004"
-      rpy="-1.5707963267949 0 -1.5707963267949" />
+      xyz="0 -0.05475 0.09675"
+      rpy="1.5708 0 0" />
     <parent
       link="pan_link" />
@@ -173,5 +173,5 @@
       link="tilt_link" />
     <axis
-      xyz="0 -1 0" />
+      xyz="0 0 1" />
   </joint>
   <transmission name="tilt_joint_trans">
@@ -184,4 +184,4 @@
     </actuator>
   </transmission>
-    </xacro:macro>
+  </xacro:macro>
 </robot>

Commit message: Fix deprecated controller types and allow basic simulation

File: poli2_description/robots/poli.urdf.xacro (robot description, xacro)
@@ -38,5 +38,4 @@
     <xacro:include filename="$(find poli2_description)/urdf/poli_components/pillar_plate.urdf.xacro"/>
     <xacro:include filename="$(find poli2_description)/urdf/poli_components/neck_mount.urdf.xacro"/>
-    <xacro:include filename="$(find poli2_description)/robots/jaco2_custom.xacro"/>
     <xacro:include filename="$(find kinova_description)/urdf/j2s7s300.xacro" />
     <xacro:property name="M_PI" value="3.14159"/>

File: poli2_description/urdf/poli_components/base_plate.urdf.xacro (robot description, xacro)
@@ -41,4 +41,9 @@
                 </geometry>
             </collision>
+            <inertial>
+                <origin xyz="0 0 0" rpy="0 0 0"/>
+                <mass value="1"/>
+                <inertia ixx="0.1" ixy="0.0" ixz="0.0" iyy="0.1" iyz="0.0" izz="0.1"/>
+            </inertial>
         </link>
     </xacro:macro>

File: poli2_description/urdf/poli_components/neck_mount.urdf.xacro (robot description, xacro)
@@ -178,5 +178,5 @@
     <type>transmission_interface/SimpleTransmission</type>
     <joint name="tilt_joint">
-      <hardwareInterface>hardware_interface/PositionJointInterface</hardwareInterface>
+      <hardwareInterface>hardware_interface/VelocityJointInterface</hardwareInterface>
     </joint>
     <actuator name="tilt_joint_actuator">

File: poli2_description/urdf/segway_components/caster_assembly.urdf.xacro (robot description, xacro)
@@ -84,8 +84,8 @@
 			<type>transmission_interface/SimpleTransmission</type>
 			<joint name="${caster_prefix}_caster_swivel">
-			    <hardwareInterface>EffortJointInterface</hardwareInterface>
+			    <hardwareInterface>hardware_interface/EffortJointInterface</hardwareInterface>
 			</joint>
 			<actuator name="${caster_prefix}_caster_swivel_motor">
-			    <hardwareInterface>EffortJointInterface</hardwareInterface>
+			    <hardwareInterface>hardware_interface/EffortJointInterface</hardwareInterface>
 				<mechanicalReduction>1</mechanicalReduction>
 			</actuator>
@@ -131,8 +131,8 @@
 			<type>transmission_interface/SimpleTransmission</type>
 			<joint name="${caster_prefix}_caster_wheel">
-			    <hardwareInterface>EffortJointInterface</hardwareInterface>
+			    <hardwareInterface>hardware_interface/EffortJointInterface</hardwareInterface>
 			</joint>
 			<actuator name="${caster_prefix}_caster_wheel_motor">
-			    <hardwareInterface>EffortJointInterface</hardwareInterface>
+			    <hardwareInterface>hardware_interface/EffortJointInterface</hardwareInterface>
 				<mechanicalReduction>1</mechanicalReduction>
 			</actuator>

Commit message: Updated Moe urdf

File: poli2_description/robots/poli.urdf.xacro (robot description, xacro)
@@ -31,10 +31,9 @@
     <xacro:include filename="$(find poli2_description)/urdf/sensors/hokuyo_ust30lx.urdf.xacro"/>
     <xacro:include filename="$(find poli2_description)/urdf/sensors/astra.urdf.xacro"/>
-    <xacro:include filename="$(find poli2_description)/urdf/sensors/sonar.urdf.xacro"/>
     <xacro:include filename="$(find poli2_description)/urdf/poli_components/base_plate.urdf.xacro"/>
     <xacro:include filename="$(find poli2_description)/urdf/poli_components/rmp_plate2.urdf.xacro"/>
     <xacro:include filename="$(find poli2_description)/urdf/poli_components/rmp_plate3.urdf.xacro"/>
     <xacro:include filename="$(find poli2_description)/urdf/poli_components/pillar.urdf.xacro"/>
-    <xacro:include filename="$(find poli2_description)/urdf/poli_components/pillar_plate.urdf.xacro"/>
+    <xacro:include filename="$(find poli2_description)/urdf/poli_components/torso.urdf.xacro"/>
     <xacro:include filename="$(find poli2_description)/urdf/poli_components/neck_mount.urdf.xacro"/>
     <xacro:include filename="$(find kinova_description)/urdf/j2s7s300.xacro" />
@@ -131,12 +130,13 @@
             <origin xyz="0.2315586 0 0.0075" rpy="0 -${HALF_PI} 0"/>
         </xacro:pillar>
-        <xacro:pillar_plate parent="pillar_telescope_link">
-            <origin xyz="-0.14899868 0.17604938 -0.14899868" rpy="0 0 0"/>
-        </xacro:pillar_plate>
-        <xacro:neck_mount parent="pillar_plate_link">
-            <origin xyz="0.2658 0.36 0.1915" rpy="-${HALF_PI} 0 0"/>
+	<!-- Torso -->
+        <xacro:torso parent="pillar_base_link">
+            <origin xyz="0.06717 -0.0308 0.06717" rpy="0 ${M_PI} 0"/>
+        </xacro:torso>
+        <xacro:neck_mount parent="torso_link">
+            <origin xyz="0 0.7125 0" rpy="-${HALF_PI} ${M_PI} 0"/>
         </xacro:neck_mount>
 	<!-- Poli Jaco Arm -->
-	<xacro:j2s7s300 base_parent="pillar_plate_link" trans="0 0.05 0.0575" rot="-${HALF_PI} -${HALF_PI} 0">
+	<xacro:j2s7s300 base_parent="torso_link" trans="0.18365 0.33377 0.14557" rot="-${HALF_PI} ${HALF_PI} 0">
 	</xacro:j2s7s300>
         <!-- Poli Sensors -->
@@ -148,9 +148,6 @@
         </xacro:hokuyo_ust10lx>
         <xacro:sensor_astra parent="tilt_link">
-	    <origin xyz="-0.22 0.0 -0.0624 " rpy="${HALF_PI} 0 ${M_PI+1.0472}"/>
+	    <origin xyz="-0.195 0.0835 0" rpy="0 0 ${HALF_PI+1.0472}"/>
         </xacro:sensor_astra>
-        <xacro:sensor_sonar parent="pillar_plate_link">
-            <origin xyz="0.007 0.022 0.203" rpy="${HALF_PI} 0 ${HALF_PI*2}"/>
-        </xacro:sensor_sonar>
     </xacro:macro>
 </robot>

File: poli2_description/urdf/poli_components/neck_mount.urdf.xacro (robot description, xacro)
@@ -22,5 +22,5 @@
 <robot xmlns:xacro="http://ros.org/wiki/xacro" name="neck_mount">
     <xacro:macro name="neck_mount" params="parent *origin">
-    <joint name="neck_base_joint" type="fixed">
+    <!--joint name="neck_base_joint" type="fixed">
             <xacro:insert_block name="origin" />
             <parent link="${parent}" />
@@ -66,5 +66,5 @@
       </geometry>
     </collision>
-   </link>
+   </link-->
    <link
     name="pan_link">
@@ -110,10 +110,7 @@
     name="pan_joint"
     type="revolute">
+    <xacro:insert_block name="origin" />
+    <parent link="${parent}" />
     <limit lower="-1.54" upper="1.54" velocity="10" effort="10"/>
-    <origin
-      xyz="0.0014145 0 0.0466"
-      rpy="0 0 0" />
-    <parent
-      link="neck_base_link" />
     <child
       link="pan_link" />
@@ -125,6 +122,6 @@
     <inertial>
       <origin
-        xyz="-0.0449449011423384 0.0505307759460616 -0.0582731595130051"
-        rpy="0 0 0" />
+        xyz="-0.0449449011423384 0 -0.0582731595130051"
+        rpy="0 1.5708 0" />
       <mass
         value="0.282648823094398" />
@@ -140,5 +137,5 @@
       <origin
         xyz="0 0 0"
-        rpy="0 0 0" />
+        rpy="0 1.5708 0.5236" />
       <geometry>
         <mesh
@@ -166,5 +163,5 @@
     <limit upper="0.0" lower="-1.0471975512" velocity="1.0" effort="10.0"/>
     <origin
-      xyz="0 -0.05475 0.09675"
+      xyz="0 0 0.095"
       rpy="1.5708 0 0" />
     <parent

File: poli2_description/urdf/poli_components/pillar.urdf.xacro (robot description, xacro)
@@ -42,26 +42,4 @@
             </collision>
         </link>
-        <joint name="pillar_telescope_joint" type="prismatic">
-            <origin xyz="0.2175586 0.1 0.02" rpy="0 -1.570796 0"/>
-            <parent link="${parent}" />
-            <child link="pillar_telescope_link" />
-            <limit effort="30" velocity="1.0" lower="0.0" upper="0.4" />
-            <axis xyz="0 1 0"/>
-        </joint>
-        <link name="pillar_telescope_link">
-            <visual>
-                <geometry>
-                    <mesh filename="package://poli2_description/meshes/components/pillar_telescope.STL" />
-                </geometry>
-                <material name="">
-                    <color rgba="0.3 0.3 0.3 1" />
-                </material>
-            </visual>
-            <collision>
-                <geometry>
-                    <mesh filename="package://poli2_description/meshes/components/pillar_telescope.STL" />
-                </geometry>
-            </collision>
-        </link>
     </xacro:macro>
 </robot>

File: poli2_description/urdf/sensors/astra.urdf.xacro (robot description, xacro)
@@ -28,5 +28,5 @@
     <link name="camera_link">
       <visual>
-        <origin xyz="-0.04 0.02 -0.01" rpy="${M_PI/2} 0 ${M_PI/2}"/>
+        <origin xyz="-0.04 0.02 0" rpy="${M_PI/2} 0 ${M_PI/2}"/>
         <geometry>
           <mesh filename="package://poli2_description/meshes/sensors/astra.dae" scale="${astra_dae_display_scale} ${astra_dae_display_scale} ${astra_dae_display_scale}"/>

Commit message: Transfer to moe1

File: poli2_description/robots/poli.urdf.xacro (robot description, xacro)
@@ -147,7 +147,12 @@
             <origin xyz="0.242 -0.015 0.33" rpy="${HALF_PI} -${HALF_PI} 0" />
         </xacro:hokuyo_ust10lx>
-        <xacro:sensor_astra parent="tilt_link">
-	    <origin xyz="-0.195 0.0835 0" rpy="0 0 ${HALF_PI+1.0472}"/>
-        </xacro:sensor_astra>
+        <link name="camera_placement_link"/>
+        <joint name="camera_placement_joint">
+            <parent name="tilt_link"/>
+            <child name="camera_placement_link"/>
+            <origin xyz="-0.195 0.0835 0" rpy="0 0 ${HALF_PI+1.0472}"/>
+        </joint>
+<!--         <xacro:sensor_astra parent="tilt_link">
+        </xacro:sensor_astra> -->
     </xacro:macro>
 </robot>
