Commit message: cleaning up launch files and xacro files

File: poli2_description/robots/moe.urdf.xacro (robot description, xacro)
@@ -1,5 +1,5 @@
 <?xml version="1.0"?>
 <robot name="segway_robot" xmlns:xacro="http://ros.org/wiki/xacro">
-  <xacro:include filename="$(find poli2_description)/robots/poli.urdf.xacro" />
+  <xacro:include filename="$(find poli2_description)/robots/poli2_segway.urdf.xacro" />
   <xacro:segway_robot />
 </robot>

File: poli2_description/robots/poli2.urdf.xacro (robot description, xacro)
@@ -148,7 +148,7 @@
         </xacro:hokuyo_ust10lx>
         <link name="camera_placement_link"/>
-        <joint name="camera_placement_joint">
-            <parent name="tilt_link"/>
-            <child name="camera_placement_link"/>
+        <joint name="camera_placement_joint" type="fixed">
+            <parent link="tilt_link"/>
+            <child link="camera_placement_link"/>
             <origin xyz="-0.195 0.0835 0" rpy="0 0 ${HALF_PI+1.0472}"/>
         </joint>
