Commit message: Cleaned up launch files for various robots

File: poli2_description/robots/barton.urdf.xacro (robot description, xacro)
@@ -1,5 +1,30 @@
 <?xml version="1.0"?>
-<robot name="freight_robot" xmlns:xacro="http://ros.org/wiki/xacro">
+<!--
+Copyright (c) 2018, The University of Texas at Austin
+All rights reserved.
+Redistribution and use in source and binary forms, with or without
+modification, are permitted provided that the following conditions are met:
+1. Redistributions of source code must retain the above copyright notice,
+   this list of conditions and the following disclaimer.
+2. Redistributions in binary form must reproduce the above copyright
+   notice, this list of conditions and the following disclaimer in the
+   documentation and/or other materials provided with the distribution.
+3. Neither the name of the copyright holder nor the names of its
+   contributors may be used to endorse or promote products derived from
+   this software without specific prior written permission.
+THIS SOFTWARE IS PROVIDED BY THE COPYRIGHT HOLDERS AND CONTRIBUTORS "AS
+IS" AND ANY EXPRESS OR IMPLIED WARRANTIES, INCLUDING, BUT NOT LIMITED TO,
+THE IMPLIED WARRANTIES OF MERCHANTABILITY AND FITNESS FOR A PARTICULAR
+PURPOSE ARE DISCLAIMED. IN NO EVENT SHALL THE COPYRIGHT HOLDER OR
+CONTRIBUTORS BE LIABLE FOR ANY DIRECT, INDIRECT, INCIDENTAL, SPECIAL,
+EXEMPLARY, OR CONSEQUENTIAL DAMAGES (INCLUDING, BUT NOT LIMITED TO,
+PROCUREMENT OF SUBSTITUTE GOODS OR SERVICES; LOSS OF USE, DATA, OR PROFITS;
+OR BUSINESS INTERRUPTION) HOWEVER CAUSED AND ON ANY THEORY OF LIABILITY,
+WHETHER IN CONTRACT, STRICT LIABILITY, OR TORT (INCLUDING NEGLIGENCE OR
+OTHERWISE) ARISING IN ANY WAY OUT OF THE USE OF THIS SOFTWARE, EVEN IF
+ADVISED OF THE POSSIBILITY OF SUCH DAMAGE.
+-->
+<robot name="barton" xmlns:xacro="http://ros.org/wiki/xacro">
   <xacro:include filename="$(find poli2_description)/robots/poli2_freight.urdf.xacro" />
-  <xacro:freight_robot />
+  <xacro:poli2_freight />
 </robot>

File: poli2_description/robots/lupe.urdf.xacro (robot description, xacro)
@@ -1,5 +1,30 @@
 <?xml version="1.0"?>
-<robot name="freight_robot" xmlns:xacro="http://ros.org/wiki/xacro">
+<!--
+Copyright (c) 2018, The University of Texas at Austin
+All rights reserved.
+Redistribution and use in source and binary forms, with or without
+modification, are permitted provided that the following conditions are met:
+1. Redistributions of source code must retain the above copyright notice,
+   this list of conditions and the following disclaimer.
+2. Redistributions in binary form must reproduce the above copyright
+   notice, this list of conditions and the following disclaimer in the
+   documentation and/or other materials provided with the distribution.
+3. Neither the name of the copyright holder nor the names of its
+   contributors may be used to endorse or promote products derived from
+   this software without specific prior written permission.
+THIS SOFTWARE IS PROVIDED BY THE COPYRIGHT HOLDERS AND CONTRIBUTORS "AS
+IS" AND ANY EXPRESS OR IMPLIED WARRANTIES, INCLUDING, BUT NOT LIMITED TO,
+THE IMPLIED WARRANTIES OF MERCHANTABILITY AND FITNESS FOR A PARTICULAR
+PURPOSE ARE DISCLAIMED. IN NO EVENT SHALL THE COPYRIGHT HOLDER OR
+CONTRIBUTORS BE LIABLE FOR ANY DIRECT, INDIRECT, INCIDENTAL, SPECIAL,
+EXEMPLARY, OR CONSEQUENTIAL DAMAGES (INCLUDING, BUT NOT LIMITED TO,
+PROCUREMENT OF SUBSTITUTE GOODS OR SERVICES; LOSS OF USE, DATA, OR PROFITS;
+OR BUSINESS INTERRUPTION) HOWEVER CAUSED AND ON ANY THEORY OF LIABILITY,
+WHETHER IN CONTRACT, STRICT LIABILITY, OR TORT (INCLUDING NEGLIGENCE OR
+OTHERWISE) ARISING IN ANY WAY OUT OF THE USE OF THIS SOFTWARE, EVEN IF
+ADVISED OF THE POSSIBILITY OF SUCH DAMAGE.
+-->
+<robot name="lupe" xmlns:xacro="http://ros.org/wiki/xacro">
   <xacro:include filename="$(find poli2_description)/robots/poli2_freight.urdf.xacro" />
-  <xacro:freight_robot />
+  <xacro:poli2_freight />
 </robot>

File: poli2_description/robots/moe.urdf.xacro (robot description, xacro)
@@ -1,5 +1,30 @@
 <?xml version="1.0"?>
-<robot name="segway_robot" xmlns:xacro="http://ros.org/wiki/xacro">
+<!--
+Copyright (c) 2018, The University of Texas at Austin
+All rights reserved.
+Redistribution and use in source and binary forms, with or without
+modification, are permitted provided that the following conditions are met:
+1. Redistributions of source code must retain the above copyright notice,
+   this list of conditions and the following disclaimer.
+2. Redistributions in binary form must reproduce the above copyright
+   notice, this list of conditions and the following disclaimer in the
+   documentation and/or other materials provided with the distribution.
+3. Neither the name of the copyright holder nor the names of its
+   contributors may be used to endorse or promote products derived from
+   this software without specific prior written permission.
+THIS SOFTWARE IS PROVIDED BY THE COPYRIGHT HOLDERS AND CONTRIBUTORS "AS
+IS" AND ANY EXPRESS OR IMPLIED WARRANTIES, INCLUDING, BUT NOT LIMITED TO,
+THE IMPLIED WARRANTIES OF MERCHANTABILITY AND FITNESS FOR A PARTICULAR
+PURPOSE ARE DISCLAIMED. IN NO EVENT SHALL THE COPYRIGHT HOLDER OR
+CONTRIBUTORS BE LIABLE FOR ANY DIRECT, INDIRECT, INCIDENTAL, SPECIAL,
+EXEMPLARY, OR CONSEQUENTIAL DAMAGES (INCLUDING, BUT NOT LIMITED TO,
+PROCUREMENT OF SUBSTITUTE GOODS OR SERVICES; LOSS OF USE, DATA, OR PROFITS;
+OR BUSINESS INTERRUPTION) HOWEVER CAUSED AND ON ANY THEORY OF LIABILITY,
+WHETHER IN CONTRACT, STRICT LIABILITY, OR TORT (INCLUDING NEGLIGENCE OR
+OTHERWISE) ARISING IN ANY WAY OUT OF THE USE OF THIS SOFTWARE, EVEN IF
+ADVISED OF THE POSSIBILITY OF SUCH DAMAGE.
+-->
+<robot name="moe" xmlns:xacro="http://ros.org/wiki/xacro">
   <xacro:include filename="$(find poli2_description)/robots/poli2_segway.urdf.xacro" />
-  <xacro:segway_robot />
+  <xacro:poli2_segway />
 </robot>

File: poli2_description/robots/poli2_freight.urdf.xacro (robot description, xacro)
@@ -20,5 +20,5 @@
 ARISING IN ANY WAY OUT OF THE USE OF THIS SOFTWARE, EVEN IF ADVISED OF THE POSSIBILITY OF SUCH DAMAGE.
 -->
-<robot name="freight_robot" xmlns:xacro="http://ros.org/wiki/xacro">
+<robot name="poli2_freight" xmlns:xacro="http://ros.org/wiki/xacro">
     <!-- Included URDF/XACRO Files -->
     <xacro:include filename="$(find poli2_description)/urdf/segway_components/battery.urdf.xacro" />

File: poli2_description/robots/poli2_segway.urdf.xacro (robot description, xacro)
@@ -20,5 +20,5 @@
 ARISING IN ANY WAY OUT OF THE USE OF THIS SOFTWARE, EVEN IF ADVISED OF THE POSSIBILITY OF SUCH DAMAGE.
 -->
-<robot name="segway_robot" xmlns:xacro="http://ros.org/wiki/xacro">
+<robot name="poli2_segway" xmlns:xacro="http://ros.org/wiki/xacro">
     <!-- Included URDF/XACRO Files -->
     <xacro:include filename="$(find poli2_description)/urdf/segway_components/battery.urdf.xacro" />
@@ -65,29 +65,29 @@
           </plugin>
         </gazebo>
-        <!-- Base link is the center of the robot's chassis between the motors projected on the ground -->
+    <!-- Base link is the center of the robot's chassis between the motors projected on the ground -->
         <link name="base_link"/>
-        <!--Chassis -->
+    <!--Chassis -->
         <xacro:powerbase_110 chassis_prefix="base" parent="base_link">
             <origin xyz="0 0 ${-wheel_vertical_offset + wheel_radius}" rpy="0 0 0" />
         </xacro:powerbase_110>
         <link name="inertial_collision_link">
-			<inertial>
-				<mass value="29.756375" />
-				<origin xyz="0.001751 0.000008 0.018544" />
-				<inertia ixx="0.696269"  ixy="0.016133" ixz="0.003232"
+            <inertial>
+                <mass value="29.756375" />
+                <origin xyz="0.001751 0.000008 0.018544" />
+                <inertia ixx="0.696269"  ixy="0.016133" ixz="0.003232"
                          iyx="0.016133"  iyy="0.299110" iyz="-0.000004"
                          izx="-0.077476" izy="-0.000004" izz="0.864394" />
-			</inertial>
+            </inertial>
             <collision>
-				<geometry>
-					<mesh filename="package://poli2_description/meshes/collision/110_powerbase_collision.stl" />
-				</geometry>
-			</collision>
-		</link>
-		<joint name="inertial_collision_joint" type="fixed" >
-		    <parent link="base_chassis_link" />
-		    <child link="inertial_collision_link" />
-		</joint>
-        <!-- Propulsion Batteries -->
+                <geometry>
+                    <mesh filename="package://poli2_description/meshes/collision/110_powerbase_collision.stl" />
+                </geometry>
+            </collision>
+        </link>
+        <joint name="inertial_collision_joint" type="fixed" >
+            <parent link="base_chassis_link" />
+            <child link="inertial_collision_link" />
+        </joint>
+    <!-- Propulsion Batteries -->
         <xacro:battery battery_prefix="mcu_1" parent="base_chassis_link">
             <origin xyz="-0.09298 0 0" rpy="0 0 0" />
@@ -97,5 +97,5 @@
             <origin xyz="0.09298 0 0" rpy="0 0 ${M_PI}" />
         </xacro:battery>
-        <!-- HMI Box -->
+    <!-- HMI Box -->
         <xacro:hmi_box_110 parent="base_chassis_link">
             <origin xyz="0 0 0.09504494" rpy="0 0 0" />
@@ -104,5 +104,5 @@
             <origin xyz="0 0 0" rpy="0 0 0" />
         </xacro:hmi_plate_110>
-        <!-- Segway wheel macros -->
+    <!-- Segway wheel macros -->
         <xacro:i2_wheel wheel_prefix="left" parent="base_chassis_link" visual_rotation="0.0">
             <origin xyz="0 ${track/2} ${wheel_vertical_offset}" rpy="0 0 0" />
@@ -111,5 +111,5 @@
             <origin xyz="0 ${-track/2} ${wheel_vertical_offset}" rpy="0 0 0" />
         </xacro:i2_wheel>
-        <!-- Segway Caster Assembly-->
+    <!-- Segway Caster Assembly-->
         <xacro:caster_assembly_110 caster_prefix="rear" parent="base_chassis_link">
             <origin xyz="-0.32784550 0 0.03326933" rpy="0 0 ${M_PI}" />
@@ -130,5 +130,5 @@
             <origin xyz="0.2315586 0 0.0075" rpy="0 -${HALF_PI} 0"/>
         </xacro:pillar>
-	<!-- Torso -->
+    <!-- Torso -->
         <xacro:torso parent="pillar_base_link">
             <origin xyz="0.06717 -0.0308 0.06717" rpy="0 ${M_PI} 0"/>
@@ -137,8 +137,8 @@
             <origin xyz="0 0.7125 0" rpy="-${HALF_PI} ${M_PI} 0"/>
         </xacro:neck_mount>
-	<!-- Poli Jaco Arm -->
-	<xacro:j2s7s300 base_parent="torso_link" trans="0.18365 0.33377 0.14557" rot="-${HALF_PI} ${HALF_PI} 0">
-	</xacro:j2s7s300>
-        <!-- Poli Sensors -->
+    <!-- Poli Jaco Arm -->
+        <xacro:j2s7s300 base_parent="torso_link" trans="0.18365 0.33377 0.14557" rot="-${HALF_PI} ${HALF_PI} 0">
+        </xacro:j2s7s300>
+    <!-- Poli Sensors -->
         <xacro:hokuyo_ust30lx laser_prefix="${REAR_LASER_PREFIX}" parent="rmp_plate2_link">
             <origin xyz="0 0.04 0.04" rpy="-${HALF_PI} -${HALF_PI} 0" />
