Commit message: Fixed mesh load warnings and simplified collision geometry

File: poli2_description/robots/poli2_segway.urdf.xacro (robot description, xacro)
@@ -122,5 +122,5 @@
         </xacro:base_plate>
         <xacro:rmp_plate2 parent="base_plate_link">
-            <origin xyz="-0.079 -0.016 0.075" rpy="0 0 0"/>
+            <origin xyz="0.165387 0.015746 0.345301" rpy="0 0 0"/>
         </xacro:rmp_plate2>
         <xacro:rmp_plate3 parent="base_plate_link">
@@ -142,5 +142,5 @@
         <!-- Poli Sensors -->
         <xacro:hokuyo_ust30lx laser_prefix="${REAR_LASER_PREFIX}" parent="rmp_plate2_link">
-            <origin xyz="0.242 0.075 0.33" rpy="-${HALF_PI} -${HALF_PI} 0" />
+            <origin xyz="0 0.04 0.04" rpy="-${HALF_PI} -${HALF_PI} 0" />
         </xacro:hokuyo_ust30lx>
         <xacro:hokuyo_ust10lx laser_prefix="${FRONT_LASER_PREFIX}" parent="rmp_plate3_link">
@@ -153,6 +153,4 @@
             <origin xyz="-0.195 0.0835 0" rpy="0 0 ${HALF_PI+1.0472}"/>
         </joint>
-<!--         <xacro:sensor_astra parent="tilt_link">
-        </xacro:sensor_astra> -->
     </xacro:macro>
 </robot>

File: poli2_description/urdf/poli_components/neck_mount.urdf.xacro (robot description, xacro)
@@ -22,49 +22,4 @@
 <robot xmlns:xacro="http://ros.org/wiki/xacro" name="neck_mount">
     <xacro:macro name="neck_mount" params="parent *origin">
-    <!--joint name="neck_base_joint" type="fixed">
-            <xacro:insert_block name="origin" />
-            <parent link="${parent}" />
-            <child link="neck_base_link" />
-            <limit effort="50" velocity="50"/>
-    </joint>
-    <link name="neck_base_link">
-    <inertial>
-      <origin
-        xyz="0.0023997 -3.3244E-06 0.033447"
-        rpy="0 0 0" />
-      <mass
-        value="0.6796" />
-      <inertia
-        ixx="0.0014012"
-        ixy="9.4856E-09"
-        ixz="-3.5218E-06"
-        iyy="0.0010212"
-        iyz="-7.8472E-10"
-        izz="0.0010421" />
-    </inertial>
-    <visual>
-      <origin
-        xyz="0 0 0"
-        rpy="0 0 0" />
-      <geometry>
-        <mesh
-          filename="package://poli2_description/meshes/components/neck/base_link.STL" />
-      </geometry>
-      <material
-        name="">
-        <color
-          rgba="0.89804 0.91765 0.92941 1" />
-      </material>
-    </visual>
-    <collision>
-      <origin
-        xyz="0 0 0"
-        rpy="0 0 0" />
-      <geometry>
-        <mesh
-          filename="package://poli2_description/meshes/components/neck/base_link.STL" />
-      </geometry>
-    </collision>
-   </link-->
    <link
     name="pan_link">
@@ -151,8 +106,8 @@
       <origin
         xyz="0 0 0"
-        rpy="0 0 0" />
+        rpy="0 1.5708 0.5236" />
       <geometry>
         <mesh
-          filename="package://poli2_description/meshes/components/neck/tilt_link.STL" />
+          filename="package://poli2_description/meshes/components/neck/tilt_link_collision.STL" />
       </geometry>
     </collision>

File: poli2_description/urdf/poli_components/pillar.urdf.xacro (robot description, xacro)
@@ -38,5 +38,5 @@
             <collision>
                 <geometry>
-                    <mesh filename="package://poli2_description/meshes/components/pillar_exterior.STL" />
+                    <mesh filename="package://poli2_description/meshes/components/pillar_exterior_collision.STL" />
                 </geometry>
             </collision>

File: poli2_description/urdf/poli_components/rmp_plate2.urdf.xacro (robot description, xacro)
@@ -38,5 +38,5 @@
             <collision>
                 <geometry>
-                    <mesh filename="package://poli2_description/meshes/components/rmp_plate2.STL" />
+                    <box size="0.298 0.006 0.189"/>
                 </geometry>
             </collision>

File: poli2_description/urdf/poli_components/torso.urdf.xacro (robot description, xacro)
@@ -57,5 +57,5 @@
             <collision>
                 <geometry>
-                    <mesh filename="package://poli2_description/meshes/components/torso_link.STL" />
+                    <mesh filename="package://poli2_description/meshes/components/torso_link_collision.STL" />
                 </geometry>
             </collision>

File: poli2_description/urdf/sensors/hokuyo_ust10lx.urdf.xacro (robot description, xacro)
@@ -35,6 +35,7 @@
             </visual>
             <collision>
+                <origin xyz="0 0 0" rpy="0 0 0" />
                 <geometry>
-                    <mesh filename="package://poli2_description/meshes/visual/sensors/hokuyo_ustlx.dae" />
+                    <box size="0.09 0.09 0.09" />
                 </geometry>
             </collision>

File: poli2_description/urdf/sensors/hokuyo_ust30lx.urdf.xacro (robot description, xacro)
@@ -35,6 +35,7 @@
             </visual>
             <collision>
+                <origin xyz="0 0 0" rpy="0 0 0" />
                 <geometry>
-                    <mesh filename="package://poli2_description/meshes/visual/sensors/hokuyo_ustlx.dae" />
+                    <box size="0.09 0.09 0.09" />
                 </geometry>
             </collision>

Commit message: Complete upgrades

File: poli2_description/robots/poli2_segway.urdf.xacro (robot description, xacro)
@@ -48,5 +48,5 @@
     <xacro:property name="wheel_length" value="0.09224900" />
     <xacro:property name="wheel_radius" value="0.2405681" />
-    <xacro:macro name="segway_robot">
+    <xacro:macro name="poli2_segway">
         <gazebo>
           <plugin name="gazebo_ros_control" filename="libgazebo_ros_control.so">

File: poli2_description/urdf/RMP_110/rmp.urdf.xacro (robot description, xacro)
@@ -21,5 +21,5 @@
 ARISING IN ANY WAY OUT OF THE USE OF THIS SOFTWARE, EVEN IF ADVISED OF THE POSSIBILITY OF SUCH DAMAGE.
 -->
-<robot name="segway_robot" xmlns:xacro="http://ros.org/wiki/xacro">
+<robot name="poli2_segway" xmlns:xacro="http://ros.org/wiki/xacro">
     <!-- Included URDF/XACRO Files -->
     <xacro:include filename="$(find poli2_description)/urdf/segway_components/battery.urdf.xacro" />
@@ -37,5 +37,5 @@
     <xacro:property name="wheel_length" value="0.09224900" />
     <xacro:property name="wheel_radius" value="0.2405681" />
-    <xacro:macro name="segway_robot">
+    <xacro:macro name="poli2_segway">
         <gazebo>
           <plugin name="gazebo_ros_control" filename="libgazebo_ros_control.so">
