Commit message: Changed macro name to match robot urdf

File: poli2_description/robots/poli2_freight.urdf.xacro (robot description, xacro)
@@ -49,5 +49,5 @@
     <xacro:property name="wheel_length" value="0.09224900" />
     <xacro:property name="wheel_radius" value="0.2405681" />
-    <xacro:macro name="freight_robot">
+    <xacro:macro name="poli2_freight">
         <gazebo>
           <plugin name="gazebo_ros_control" filename="libgazebo_ros_control.so">

Commit message: static transform to allign pointcloud with moveit RobotModel (rough and ugly)

File: poli2_description/robots/poli2_freight.urdf.xacro (robot description, xacro)
@@ -76,5 +76,5 @@
         </xacro:torso>
         <xacro:neck_mount parent="torso_link">
-            <origin xyz="0 0.7125 0" rpy="-${HALF_PI} ${M_PI} 0"/>
+            <origin xyz="0 0.7125 0" rpy="-1.57 0 0"/>
         </xacro:neck_mount>
 	<!-- Poli Jaco Arm -->

File: poli2_description/urdf/poli_components/neck_mount.urdf.xacro (robot description, xacro)
@@ -162,6 +162,4 @@
         xyz="0 0 0"
         rpy="0 0 0" />
-      <geometry>
-        <mesh
           filename="package://moxi_description/meshes/components/collision_tilt_link.STL"/>
       </geometry>
@@ -223,5 +221,5 @@
       <geometry>
         <mesh
-          filename="package://moxi_description/meshes/components/head_shell_link.STL" />
+          filename="package://poli2_description/meshes/components/Moxi_Tufts_Head.stl" />
       </geometry>
       <material
